Commit message: [resources] fixed rotation of kitchen island

File: resources/kitchen.urdf (robot description, URDF)
Before this commit: robot iai_oven_area, 84 links, 83 joints
Joints:
- joint kitchen_island_footprint_joint: origin xyz=-1.365 0.59 0 rpy=0 0 1 -> xyz=-1.365 0.59 0 rpy=0 0 0

Commit message: [Refactor] Refactored urdfs, orm classes and formatting to produce no warnings anymore.

File: resources/kitchen.urdf (robot description, URDF)
Before this commit: robot iai_oven_area, 84 links, 83 joints
Joints:
- joint sink_area_dish_washer_main_joint: axis (none) -> 1 0 0

File: resources/pr2.urdf (robot description, URDF)
Before this commit: robot pr2, 88 links, 87 joints
Links:
- link wide_stereo_optical_frame: mass None -> 0.1
