Commit message: Fix tiago_dual

File: resources/tiago_dual.urdf (robot description, URDF)
Before this commit: robot tiago_dual, 69 links, 68 joints
Links:
- link arm_left_1_link: mass 1.563428 -> None; geometry collision mesh filename=package://pycram/resources/tiago_dual/stl/arm_1_collision.s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 scale=1.0 1.0000000000000004 1.0000000000000004
- link arm_left_2_link: mass 1.800397 -> None; geometry collision mesh filename=package://pycram/resources/tiago_dual/stl/arm_2_collision.s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 scale=-0.9999999999999996 1.0 0.9999999999999996
- link arm_left_3_link: mass 1.8 -> None; geometry collision mesh filename=package://pycram/resources/tiago_dual/stl/arm_3_collision.s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 scale=-0.9999999999999996 1.0 0.9999999999999996
- link arm_left_4_link: mass 1.432697 -> None; geometry collision mesh filename=package://pycram/resources/tiago_dual/stl/arm_4_collision.s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 scale=0.9999999999999996 0.9999999999999996 -1.0
- link arm_left_5_link: mass 0.9359143689 -> None; geometry collision mesh filename=package://pycram/resources/tiago_dual/stl/arm_5_collision_w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 scale=0.9999999999999996 0.9999999999999996 -1.0
- link arm_left_6_link: mass 0.30275767222 -> None; geometry collision mesh filename=package://pycram/resources/tiago_dual/stl/arm_6_collision_w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 scale=0.9999999999999996 -0.9999999999999996 1.0
- link arm_left_7_link: mass 0.1 -> None
- link arm_left_tool_link: mass 0.1 -> None; geometry collision cylinder length=0.005 radius=0.005
- link arm_right_1_link: mass 1.563428 -> None; geometry collision mesh filename=package://pycram/resources/tiago_dual/stl/arm_1_collision.s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 scale=-0.9999999999999996 0.9999999999999996 1.0
- link arm_right_2_link: mass 1.800397 -> None; geometry collision mesh filename=package://pycram/resources/tiago_dual/stl/arm_2_collision.s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 scale=1.0 1.0 1.0
- link arm_right_3_link: mass 1.8 -> None; geometry collision mesh filename=package://pycram/resources/tiago_dual/stl/arm_3_collision.s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 scale=1.0 1.0 1.0
- link arm_right_4_link: mass 1.432697 -> None; geometry collision mesh filename=package://pycram/resources/tiago_dual/stl/arm_4_collision.s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 scale=1.0 1.0 1.0
- link arm_right_5_link: mass 0.9359143689 -> None; geometry collision mesh filename=package://pycram/resources/tiago_dual/stl/arm_5_collision_w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 scale=1.0 1.0 1.0
- link arm_right_6_link: mass 0.30275767222 -> None; geometry collision mesh filename=package://pycram/resources/tiago_dual/stl/arm_6_collision_w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 scale=1.0 1.0 1.0
- link arm_right_7_link: mass 0.1 -> None
- link arm_right_tool_link: mass 0.1 -> None; geometry collision cylinder length=0.005 radius=0.005
- link base_antenna_left_link: mass 1e-06 -> None; geometry collision cylinder length=0.17 radius=0.005
- link base_antenna_right_link: mass 1e-06 -> None; geometry collision cylinder length=0.17 radius=0.005
- link base_cover_link: mass 0.25821 -> None; geometry 
- link base_imu_link: mass 0.01 -> None
- link base_laser_link: mass 0.28922 -> None; geometry 
- link base_link: mass 28.26649 -> None; geometry collision mesh filename=package://pycram/resources/tiago_dual/stl/base_collision.stl scale=1.0 1.0 1.0
- link base_sonar_01_link: mass 0.001 -> None; geometry 
- link base_sonar_02_link: mass 0.001 -> None; geometry 
- link base_sonar_03_link: mass 0.001 -> None; geometry 
- link caster_back_left_1_link: mass 0.05144761 -> None; geometry 
- link caster_back_left_2_link: mass 0.08855784 -> None; geometry collision sphere radius=0.025
- link caster_back_right_1_link: mass 0.05144761 -> None; geometry 
- link caster_back_right_2_link: mass 0.08855784 -> None; geometry collision sphere radius=0.025
- link caster_front_left_1_link: mass 0.05144761 -> None; geometry 
- link caster_front_left_2_link: mass 0.08855784 -> None; geometry collision sphere radius=0.025
- link caster_front_right_1_link: mass 0.05144761 -> None; geometry 
- link caster_front_right_2_link: mass 0.08855784 -> None; geometry collision sphere radius=0.025
- link gripper_left_grasping_frame: mass 0.0001 -> None
- link gripper_left_left_finger_link: mass 0.10998 -> None; geometry collision box size=0.010000000000000002 0.05 0.11
- link gripper_left_link: mass 0.60266 -> None; geometry collision mesh filename=package://pycram/resources/tiago_dual/stl/gripper_link_coll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 scale=1.0 1.0 1.0
- link gripper_left_right_finger_link: mass 0.10998 -> None; geometry collision box size=0.010000000000000002 0.05 0.11
- link gripper_left_tool_link: mass 0.0001 -> None
- link gripper_right_grasping_frame: mass 0.0001 -> None
- link gripper_right_left_finger_link: mass 0.10998 -> None; geometry collision box size=0.010000000000000002 0.05 0.11
- link gripper_right_link: mass 0.60266 -> None; geometry collision mesh filename=package://pycram/resources/tiago_dual/stl/gripper_link_coll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 scale=1.0 1.0 1.0
- link gripper_right_right_finger_link: mass 0.10998 -> None; geometry collision box size=0.010000000000000002 0.05 0.11
- link gripper_right_tool_link: mass 0.0001 -> None
- link head_1_link: mass 0.6222 -> None; geometry collision mesh filename=package://pycram/resources/tiago_dual/stl/head_1_collision.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 scale=1.0 1.0 1.0
- link head_2_link: mass 0.66123 -> None; geometry collision mesh filename=package://pycram/resources/tiago_dual/stl/head_2_collision.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 scale=1.0 1.0 1.0
- link rgbd_laser_link: mass 0.0001 -> None
- link suspension_left_link: mass 10.0 -> None
- link suspension_right_link: mass 10.0 -> None
- link torso_fixed_column_link: mass 0.01 -> None; geometry collision box size=0.23 0.23 0.55
- link torso_fixed_link: mass 14.0136 -> None; geometry collision box size=0.25 0.25 0.1; collision box size=0.4 0.25 0.04
- link torso_lift_link: mass 9.594213 -> None; geometry collision mesh filename=package://pycram/resources/tiago_dual/stl/torso_lift_collis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 scale=1.0 1.0 1.0; collision mesh filename=package://pycram/resources/tiago_dual/stl/torso_lift_collis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 scale=1.0 1.0 1.0
- link wheel_left_link: mass 1.82362 -> None; geometry collision sphere radius=0.0985
- link wheel_right_link: mass 1.82362 -> None; geometry collision sphere radius=0.0985
- link wrist_left_ft_link: mass 0.1 -> None; geometry collision cylinder length=0.0157 radius=0.0225
- link wrist_left_ft_tool_link: mass 0.1 -> None; geometry collision cylinder length=0.00975 radius=0.025
- link wrist_right_ft_link: mass 0.1 -> None; geometry collision cylinder length=0.0157 radius=0.0225
- link wrist_right_ft_tool_link: mass 0.1 -> None; geometry collision cylinder length=0.00975 radius=0.025
- link xtion_depth_frame: mass 0.001 -> None
- link xtion_depth_optical_frame: mass 0.001 -> None
- link xtion_link: mass 0.2197 -> None
- link xtion_optical_frame: mass 0.001 -> None
- link xtion_orbbec_aux_joint_frame: mass 0.001 -> None
- link xtion_rgb_frame: mass 0.001 -> None
- link xtion_rgb_optical_frame: mass 0.001 -> None
Joints:
- removed joint arm_left_tool_joint
- removed joint arm_right_tool_joint
- removed joint base_antenna_left_joint
- removed joint base_antenna_right_joint
- removed joint base_footprint_joint
- removed joint base_imu_joint
- removed joint base_laser_joint
- removed joint base_mic_back_left_joint
- removed joint base_mic_back_right_joint
- removed joint base_mic_front_left_joint
- removed joint base_mic_front_right_joint
- removed joint base_sonar_01_joint
- removed joint base_sonar_02_joint
- removed joint base_sonar_03_joint
- removed joint cover_joint
- removed joint gripper_left_joint
- removed joint gripper_left_tool_joint
- removed joint gripper_right_joint
- removed joint gripper_right_tool_joint
- removed joint rgbd_laser_joint
- removed joint torso_fixed_column_joint
- removed joint torso_fixed_joint
- removed joint wrist_left_ft_joint
- removed joint wrist_left_tool_joint
- removed joint wrist_right_ft_joint
- removed joint wrist_right_tool_joint
- removed joint xtion_depth_joint
- removed joint xtion_depth_optical_joint
- removed joint xtion_joint
- removed joint xtion_optical_joint
- removed joint xtion_orbbec_aux_joint
- removed joint xtion_rgb_joint
- removed joint xtion_rgb_optical_joint
- added joint arm_left_tool_link_joint: type fixed, parent arm_left_7_link, child arm_left_tool_link, origin xyz=0.0 0.0 -0.046 rpy=-1.5707963267948968 1.5707963267948963 0.0
- added joint arm_right_tool_link_joint: type fixed, parent arm_right_7_link, child arm_right_tool_link, origin xyz=0.0 0.0 0.046 rpy=-1.570796326794897 -1.5707963267948966 0.0
- added joint base_antenna_left_link_joint: type fixed, parent base_link, child base_antenna_left_link, origin xyz=-0.201 0.1062 0.195 rpy=0.0 -0.0 0.0
- added joint base_antenna_right_link_joint: type fixed, parent base_link, child base_antenna_right_link, origin xyz=-0.201 -0.1062 0.195 rpy=0.0 -0.0 0.0
- added joint base_cover_link_joint: type fixed, parent base_footprint, child base_cover_link, origin xyz=0.0 0.0 0.13 rpy=0.0 -0.0 0.0
- added joint base_imu_link_joint: type fixed, parent base_link, child base_imu_link, origin xyz=0.10171 0.0 0.11282 rpy=0.0 0.0 -1.5707963267948966
- added joint base_laser_link_joint: type fixed, parent base_link, child base_laser_link, origin xyz=0.202 0.0 -0.004 rpy=0.0 -0.0 0.0
- added joint base_link_joint: type fixed, parent base_footprint, child base_link, origin xyz=0.0 0.0 0.0985 rpy=0.0 -0.0 0.0
- added joint base_mic_back_left_link_joint: type fixed, parent base_link, child base_mic_back_left_link, origin xyz=-0.1082 -0.0599 0.195 rpy=0.0 -0.0 0.0
- added joint base_mic_back_right_link_joint: type fixed, parent base_link, child base_mic_back_right_link, origin xyz=-0.1082 -0.13789 0.195 rpy=0.0 -0.0 0.0
- added joint base_mic_front_left_link_joint: type fixed, parent base_link, child base_mic_front_left_link, origin xyz=0.23182 0.03902 0.195 rpy=0.0 -0.0 0.0
- added joint base_mic_front_right_link_joint: type fixed, parent base_link, child base_mic_front_right_link, origin xyz=0.23182 -0.03902 0.195 rpy=0.0 -0.0 0.0
- added joint base_sonar_01_link_joint: type fixed, parent base_link, child base_sonar_01_link, origin xyz=-0.183 -0.183 0.173 rpy=0.0 -0.0 -2.356194490192345
- added joint base_sonar_02_link_joint: type fixed, parent base_link, child base_sonar_02_link, origin xyz=-0.259 0.0 0.173 rpy=0.0 -0.0 3.141592653589793
- added joint base_sonar_03_link_joint: type fixed, parent base_link, child base_sonar_03_link, origin xyz=-0.183 0.183 0.173 rpy=0.0 -0.0 2.356194490192345
- added joint gripper_left_link_joint: type fixed, parent wrist_left_ft_tool_link, child gripper_left_link, origin xyz=0.01 0.0 0.0 rpy=3.141592653589793 1.5707963267948966 0.0
- added joint gripper_left_tool_link_joint: type fixed, parent wrist_left_ft_tool_link, child gripper_left_tool_link, origin xyz=0.01 0.0 0.0 rpy=3.141592653589793 1.5707963267948966 0.0
- added joint gripper_right_link_joint: type fixed, parent wrist_right_ft_tool_link, child gripper_right_link, origin xyz=0.01 0.0 0.0 rpy=3.141592653589793 1.5707963267948966 0.0
- added joint gripper_right_tool_link_joint: type fixed, parent wrist_right_ft_tool_link, child gripper_right_tool_link, origin xyz=0.01 0.0 0.0 rpy=3.141592653589793 1.5707963267948966 0.0
- added joint rgbd_laser_link_joint: type fixed, parent base_footprint, child rgbd_laser_link, origin xyz=-0.9 0.0 0.0 rpy=0.0 -0.0 0.0
- added joint torso_fixed_column_link_joint: type fixed, parent base_link, child torso_fixed_column_link, origin xyz=-0.062 0.0 0.195 rpy=0.0 -0.0 0.0
- added joint torso_fixed_link_joint: type fixed, parent base_link, child torso_fixed_link, origin xyz=-0.062 0.0 0.193 rpy=0.0 -0.0 0.0
- added joint wrist_left_ft_link_joint: type fixed, parent arm_left_tool_link, child wrist_left_ft_link, origin xyz=0.00785 0.0 0.0 rpy=1.5707963267948966 -0.0 1.5707963267948966
- added joint wrist_left_ft_tool_link_joint: type fixed, parent wrist_left_ft_link, child wrist_left_ft_tool_link, origin xyz=0.0 0.0 0.012725 rpy=-1.5707963267948966 -1.5707963267948966 0.0
- added joint wrist_right_ft_link_joint: type fixed, parent arm_right_tool_link, child wrist_right_ft_link, origin xyz=0.00785 0.0 0.0 rpy=1.5707963267948966 -0.0 1.5707963267948966
- added joint wrist_right_ft_tool_link_joint: type fixed, parent wrist_right_ft_link, child wrist_right_ft_tool_link, origin xyz=0.0 0.0 0.012725 rpy=-1.5707963267948966 -1.5707963267948966 0.0
- added joint xtion_depth_frame_joint: type fixed, parent xtion_rgb_frame, child xtion_depth_frame, origin xyz=0.0 0.025 0.0 rpy=0.0 -0.0 0.0
- added joint xtion_depth_optical_frame_joint: type fixed, parent xtion_depth_frame, child xtion_depth_optical_frame, origin xyz=0.0 0.0 0.0 rpy=-1.5707963267948966 -0.0 -1.5707963267948966
- added joint xtion_link_joint: type fixed, parent head_2_link, child xtion_link, origin xyz=0.0908 0.08 0.0 rpy=-1.5707963267948966 0.0 0.0
- added joint xtion_optical_frame_joint: type fixed, parent xtion_link, child xtion_optical_frame, origin xyz=0.0 0.0 0.0 rpy=-1.5707963267948966 -0.0 -1.5707963267948966
- added joint xtion_orbbec_aux_joint_frame_joint: type fixed, parent xtion_link, child xtion_orbbec_aux_joint_frame, origin xyz=0.0 0.0 0.0 rpy=0.0 -0.0 0.0
- added joint xtion_rgb_frame_joint: type fixed, parent xtion_orbbec_aux_joint_frame, child xtion_rgb_frame, origin xyz=0.0 0.022 0.0 rpy=0.0 -0.0 0.0
- added joint xtion_rgb_optical_frame_joint: type fixed, parent xtion_rgb_frame, child xtion_rgb_optical_frame, origin xyz=0.0 0.0 0.0 rpy=-1.5707963267948966 -0.0 -1.5707963267948966
- joint arm_left_1_joint: axis 0.0 0.0 1.0 -> 0 0 1; limit lower=-1.1780972450961724 upper=1.5707963267948966 effort=43.0 velocity=1.95 -> lower=-1.1780972450961724 upper=1.5707963267948966 effort=1000 velocity=1000; origin xyz=0.02556 0.19 -0.171 rpy=3.141592653589793 0.0 1.5707963267948966 -> xyz=0.02556000091135502 0.1899999976158142 -0.17100000381469727 rpy=3.141592653589793 -0.0 1.5707963267948966
- joint arm_left_2_joint: axis 0.0 0.0 1.0 -> 0 0 1; limit lower=-1.1780972450961724 upper=1.5707963267948966 effort=43.0 velocity=1.95 -> lower=-1.1780972450961724 upper=1.5707963267948966 effort=1000 velocity=1000; origin xyz=0.125 -0.0195 0.031 rpy=1.5707963267948966 0.0 0.0 -> xyz=0.125 -0.019500000402331352 0.03099999949336052 rpy=1.5707963267948966 0.0 0.0
- joint arm_left_3_joint: axis 0.0 0.0 1.0 -> 0 0 1; limit lower=-0.7853981633974483 upper=3.9269908169872414 effort=26.0 velocity=2.35 -> lower=-0.7853981633974483 upper=3.9269908169872414 effort=1000 velocity=1000; origin xyz=0.0895 0.0 -0.0015 rpy=-1.5707963267948966 3.141592653589793 -1.5707963267948966 -> xyz=0.08950000256299973 3.0814879110195774e-33 -0.001500000013038516 rpy=1.5707963267948968 -0.0 1.5707963267948968
- joint arm_left_4_joint: axis 0.0 0.0 1.0 -> 0 0 1; limit lower=-0.39269908169872414 upper=2.356194490192345 effort=26.0 velocity=2.35 -> lower=-0.39269908169872414 upper=2.356194490192345 effort=1000 velocity=1000; origin xyz=-0.02 -0.027 0.222 rpy=1.5707963267948966 -1.5707963267948966 0.0 -> xyz=-0.019999999552965164 -0.027000000700354576 0.22200000286102295 rpy=1.5707963267948968 -1.5707963267948963 0.0
- joint arm_left_5_joint: axis 0.0 0.0 1.0 -> 0 0 1; limit lower=-2.0943951023931953 upper=2.0943951023931953 effort=3.0 velocity=1.95 -> lower=-2.0943951023931953 upper=2.0943951023931953 effort=1000 velocity=1000; origin xyz=0.162 -0.02 -0.027 rpy=1.5707963267948966 -1.5707963267948966 -1.5707963267948966 -> xyz=0.16200000047683716 -0.019999999552965164 -0.027000000700354576 rpy=-0.0 -1.5707963267948966 0.0
- joint arm_left_6_joint: axis 0.0 0.0 1.0 -> 0 0 1; limit lower=-1.413716694115407 upper=1.413716694115407 effort=6.6 velocity=1.76 -> lower=-1.413716694115407 upper=1.413716694115407 effort=1000 velocity=1000; origin xyz=0.0 0.0 -0.15 rpy=0.0 -1.5707963267948966 -1.5707963267948966 -> xyz=0.0 0.0 -0.15000000596046448 rpy=-1.5707963267948968 -1.5707963267948963 0.0
- joint arm_left_7_joint: axis 0.0 0.0 1.0 -> 0 0 1; limit lower=-2.0943951023931953 upper=2.0943951023931953 effort=6.6 velocity=1.76 -> lower=-2.0943951023931953 upper=2.0943951023931953 effort=1000 velocity=1000; origin xyz=0.0 0.0 0.0 rpy=1.5707963267948966 0.0 1.5707963267948966 -> xyz=0.0 0.0 0.0 rpy=1.5707963267948968 -0.0 1.5707963267948968
- joint arm_right_1_joint: axis 0.0 0.0 1.0 -> 0 0 1; limit lower=-1.1780972450961724 upper=1.5707963267948966 effort=43.0 velocity=1.95 -> lower=-1.1780972450961724 upper=1.5707963267948966 effort=1000 velocity=1000; origin xyz=0.02556 -0.19 -0.171 rpy=0.0 0.0 -1.5707963267948966 -> xyz=0.02556000091135502 -0.1899999976158142 -0.17100000381469727 rpy=0.0 0.0 -1.5707963267948966
- joint arm_right_2_joint: axis 0.0 0.0 1.0 -> 0 0 1; limit lower=-1.1780972450961724 upper=1.5707963267948966 effort=43.0 velocity=1.95 -> lower=-1.1780972450961724 upper=1.5707963267948966 effort=1000 velocity=1000; origin xyz=0.125 -0.0195 -0.031 rpy=-1.5707963267948966 0.0 0.0 -> xyz=0.125 -0.019500000402331352 -0.03099999949336052 rpy=-1.5707963267948966 0.0 0.0
- joint arm_right_3_joint: axis 0.0 0.0 1.0 -> 0 0 1; limit lower=-0.7853981633974483 upper=3.9269908169872414 effort=26.0 velocity=2.35 -> lower=-0.7853981633974483 upper=3.9269908169872414 effort=1000 velocity=1000; origin xyz=0.0895 0.0 -0.0015 rpy=-1.5707963267948966 0.0 1.5707963267948966 -> xyz=0.08950000256299973 0.0 -0.001500000013038516 rpy=-1.5707963267948968 -0.0 1.5707963267948968
- joint arm_right_4_joint: axis 0.0 0.0 1.0 -> 0 0 1; limit lower=-0.39269908169872414 upper=2.356194490192345 effort=26.0 velocity=2.35 -> lower=-0.39269908169872414 upper=2.356194490192345 effort=1000 velocity=1000; origin xyz=-0.02 -0.027 -0.222 rpy=-1.5707963267948966 -1.5707963267948966 0.0 -> xyz=-0.019999999552965164 -0.027000000700354576 -0.22200000286102295 rpy=-1.5707963267948968 -1.5707963267948963 0.0
- joint arm_right_5_joint: axis 0.0 0.0 1.0 -> 0 0 1; limit lower=-2.0943951023931953 upper=2.0943951023931953 effort=3.0 velocity=1.95 -> lower=-2.0943951023931953 upper=2.0943951023931953 effort=1000 velocity=1000; origin xyz=-0.162 0.02 0.027 rpy=1.5707963267948966 -1.5707963267948966 -1.5707963267948966 -> xyz=-0.16200000047683716 0.019999999552965164 0.027000000700354576 rpy=-0.0 -1.5707963267948966 0.0
- joint arm_right_6_joint: axis 0.0 0.0 1.0 -> 0 0 1; limit lower=-1.413716694115407 upper=1.413716694115407 effort=6.6 velocity=1.76 -> lower=-1.413716694115407 upper=1.413716694115407 effort=1000 velocity=1000; origin xyz=0.0 0.0 0.15 rpy=0.0 -1.5707963267948966 -1.5707963267948966 -> xyz=-0.0 -0.0 0.15000000596046448 rpy=-1.5707963267948968 -1.5707963267948963 0.0
- joint arm_right_7_joint: axis 0.0 0.0 1.0 -> 0 0 1; limit lower=-2.0943951023931953 upper=2.0943951023931953 effort=6.6 velocity=1.76 -> lower=-2.0943951023931953 upper=2.0943951023931953 effort=1000 velocity=1000; origin xyz=0.0 0.0 0.0 rpy=1.5707963267948966 0.0 1.5707963267948966 -> xyz=0.0 0.0 0.0 rpy=1.5707963267948968 -0.0 1.5707963267948968
- joint caster_back_left_1_joint: axis 0.0 0.0 1.0 -> 0 0 1; origin xyz=-0.17350000000000002 0.102 -0.0335 rpy=0.0 0.0 0.0 -> xyz=-0.17350000143051147 0.10199999809265137 -0.03350000083446503 rpy=0.0 -0.0 0.0
- joint caster_back_left_2_joint: axis 0.0 0.0 1.0 -> 0 0 1; origin xyz=-0.016 0.0 -0.04 rpy=-1.5707963267948966 0.0 0.0 -> xyz=-0.01600000075995922 0.0 -0.03999999910593033 rpy=-1.5707963267948966 0.0 0.0
- joint caster_back_right_1_joint: axis 0.0 0.0 1.0 -> 0 0 1; origin xyz=-0.17350000000000002 -0.102 -0.0335 rpy=0.0 0.0 0.0 -> xyz=-0.17350000143051147 -0.10199999809265137 -0.03350000083446503 rpy=0.0 -0.0 0.0
- joint caster_back_right_2_joint: axis 0.0 0.0 1.0 -> 0 0 1; origin xyz=-0.016 0.0 -0.04 rpy=-1.5707963267948966 0.0 0.0 -> xyz=-0.01600000075995922 0.0 -0.03999999910593033 rpy=-1.5707963267948966 0.0 0.0
- joint caster_front_left_1_joint: axis 0.0 0.0 1.0 -> 0 0 1; origin xyz=0.1695 0.102 -0.0335 rpy=0.0 0.0 0.0 -> xyz=0.16949999332427979 0.10199999809265137 -0.03350000083446503 rpy=0.0 -0.0 0.0
- joint caster_front_left_2_joint: axis 0.0 0.0 1.0 -> 0 0 1; origin xyz=-0.016 0.0 -0.04 rpy=-1.5707963267948966 0.0 0.0 -> xyz=-0.01600000075995922 0.0 -0.03999999910593033 rpy=-1.5707963267948966 0.0 0.0
- joint caster_front_right_1_joint: axis 0.0 0.0 1.0 -> 0 0 1; origin xyz=0.1695 -0.102 -0.0335 rpy=0.0 0.0 0.0 -> xyz=0.16949999332427979 -0.10199999809265137 -0.03350000083446503 rpy=0.0 -0.0 0.0
- joint caster_front_right_2_joint: axis 0.0 0.0 1.0 -> 0 0 1; origin xyz=-0.016 0.0 -0.04 rpy=-1.5707963267948966 0.0 0.0 -> xyz=-0.01600000075995922 0.0 -0.03999999910593033 rpy=-1.5707963267948966 0.0 0.0
- joint gripper_left_grasping_frame_joint: origin xyz=0.0 0.0 -0.12 rpy=-1.5708 1.5708 0.0 -> xyz=0.0 0.0 -0.12 rpy=1.5707926535159558 1.5707926535897936 3.1415926535595684
- joint gripper_left_left_finger_joint: axis -1.0 0.0 0.0 -> -1 0 0; limit lower=0.0 upper=0.045 effort=16.0 velocity=0.05 -> lower=0.0 upper=0.04500000178813934 effort=1000 velocity=1000; origin xyz=0.0 0.0 0.0 rpy=0.0 0.0 0.0 -> xyz=0.0 -6.162975822039155e-33 0.0 rpy=1.3454695115200456e-32 3.316838427515549e-64 -4.930380657631325e-32
- joint gripper_left_right_finger_joint: axis 1.0 0.0 0.0 -> 1 0 0; limit lower=0.0 upper=0.045 effort=16.0 velocity=0.05 -> lower=0.0 upper=0.04500000178813934 effort=1000 velocity=1000; origin xyz=0.0 0.0 0.0 rpy=0.0 0.0 0.0 -> xyz=0.0 -6.162975822039155e-33 0.0 rpy=1.3454695115200456e-32 3.316838427515549e-64 -4.930380657631325e-32
- joint gripper_right_grasping_frame_joint: origin xyz=0.0 0.0 -0.12 rpy=-1.5708 1.5708 0.0 -> xyz=0.0 0.0 -0.12 rpy=1.5707926535159558 1.5707926535897936 3.1415926535595684
- joint gripper_right_left_finger_joint: axis -1.0 0.0 0.0 -> -1 0 0; limit lower=0.0 upper=0.045 effort=16.0 velocity=0.05 -> lower=0.0 upper=0.04500000178813934 effort=1000 velocity=1000; origin xyz=0.0 0.0 0.0 rpy=0.0 0.0 0.0 -> xyz=0.0 0.0 0.0 rpy=-2.9907775833605145e-33 1.8432089935347544e-65 1.2325951644078312e-32
- joint gripper_right_right_finger_joint: axis 1.0 0.0 0.0 -> 1 0 0; limit lower=0.0 upper=0.045 effort=16.0 velocity=0.05 -> lower=0.0 upper=0.04500000178813934 effort=1000 velocity=1000; origin xyz=0.0 0.0 0.0 rpy=0.0 0.0 0.0 -> xyz=0.0 0.0 0.0 rpy=-2.9907775833605145e-33 1.8432089935347544e-65 1.2325951644078312e-32
- joint head_1_joint: axis 0.0 0.0 1.0 -> 0 0 1; limit lower=-1.3089969389957472 upper=1.3089969389957472 effort=5.197 velocity=3.0 -> lower=-1.3089969389957472 upper=1.3089969389957472 effort=1000 velocity=1000; origin xyz=0.182 0.0 0.0 rpy=0.0 0.0 0.0 -> xyz=0.18199999630451202 0.0 0.0 rpy=0.0 -0.0 0.0
- joint head_2_joint: axis 0.0 0.0 1.0 -> 0 0 1; limit lower=-1.0471975511965976 upper=0.7853981633974483 effort=2.77 velocity=3.0 -> lower=-1.0471975511965976 upper=0.7853981633974483 effort=1000 velocity=1000; origin xyz=0.005 0.0 0.098 rpy=1.5707963267948966 0.0 0.0 -> xyz=0.004999999888241291 0.0 0.09799999743700027 rpy=1.5707963267948966 -0.0 0.0
- joint suspension_left_joint: axis 0.0 0.0 1.0 -> 0 0 1; limit lower=-0.005 upper=0.005 effort=100.0 velocity=1.0 -> lower=-0.004999999888241291 upper=0.004999999888241291 effort=1000 velocity=1000; origin xyz=0.0 0.0 0.0 rpy=0.0 0.0 0.0 -> xyz=0.0 0.0 0.0 rpy=0.0 -0.0 0.0
- joint suspension_right_joint: axis 0.0 0.0 1.0 -> 0 0 1; limit lower=-0.005 upper=0.005 effort=100.0 velocity=1.0 -> lower=-0.004999999888241291 upper=0.004999999888241291 effort=1000 velocity=1000; origin xyz=0.0 0.0 0.0 rpy=0.0 0.0 0.0 -> xyz=0.0 0.0 0.0 rpy=0.0 -0.0 0.0
- joint torso_lift_joint: axis 0.0 0.0 1.0 -> 0 0 1; limit lower=0.0 upper=0.35 effort=2000.0 velocity=0.07 -> lower=0.0 upper=0.3499999940395355 effort=1000 velocity=1000; origin xyz=0.0 0.0 0.597 rpy=0.0 0.0 0.0 -> xyz=0.0 0.0 0.597000002861023 rpy=0.0 -0.0 0.0
- joint wheel_left_joint: axis 0.0 0.0 1.0 -> 0 0 1; limit lower=0 upper=0 effort=6.0 velocity=10.152284263959391 -> (none); origin xyz=0.0 0.2022 0.0 rpy=-1.5707963267948966 0.0 0.0 -> xyz=0.0 0.2021999955177307 0.0 rpy=-1.5707963267948966 0.0 0.0
- joint wheel_right_joint: axis 0.0 0.0 1.0 -> 0 0 1; limit lower=0 upper=0 effort=6.0 velocity=10.152284263959391 -> (none); origin xyz=0.0 -0.2022 0.0 rpy=-1.5707963267948966 0.0 0.0 -> xyz=0.0 -0.2021999955177307 0.0 rpy=-1.5707963267948966 0.0 0.0
