Commit message: Convert pr2

File: resources/pr2.urdf (robot description, URDF)
Before this commit: robot pr2, 88 links, 87 joints
Links:
- link base_bellow_link: mass 1.0 -> None; geometry collision box size=0.05 0.37 0.3
- link base_footprint: mass 1.0 -> None; geometry 
- link base_laser_link: mass 0.001 -> None
- link base_link: mass 116.0 -> None; geometry collision mesh filename=package://pycram/resources/pr2/stl/base_L.stl scale=1.0 1.0 1.0
- link bl_caster_l_wheel_link: mass 0.44036 -> None; geometry collision cylinder length=0.034 radius=0.074792
- link bl_caster_r_wheel_link: mass 0.44036 -> None; geometry collision cylinder length=0.034 radius=0.074792
- link bl_caster_rotation_link: mass 3.473082 -> None; geometry collision mesh filename=package://pycram/resources/pr2/stl/caster_L.stl scale=1.0 1.0 1.0
- link br_caster_l_wheel_link: mass 0.44036 -> None; geometry collision cylinder length=0.034 radius=0.074792
- link br_caster_r_wheel_link: mass 0.44036 -> None; geometry collision cylinder length=0.034 radius=0.074792
- link br_caster_rotation_link: mass 3.473082 -> None; geometry collision mesh filename=package://pycram/resources/pr2/stl/caster_L.stl scale=1.0 1.0 1.0
- link double_stereo_link: mass 0.1 -> None; geometry 
- link fl_caster_l_wheel_link: mass 0.44036 -> None; geometry collision cylinder length=0.034 radius=0.074792
- link fl_caster_r_wheel_link: mass 0.44036 -> None; geometry collision cylinder length=0.034 radius=0.074792
- link fl_caster_rotation_link: mass 3.473082 -> None; geometry collision mesh filename=package://pycram/resources/pr2/stl/caster_L.stl scale=1.0 1.0 1.0
- link fr_caster_l_wheel_link: mass 0.44036 -> None; geometry collision cylinder length=0.034 radius=0.074792
- link fr_caster_r_wheel_link: mass 0.44036 -> None; geometry collision cylinder length=0.034 radius=0.074792
- link fr_caster_rotation_link: mass 3.473082 -> None; geometry collision mesh filename=package://pycram/resources/pr2/stl/caster_L.stl scale=1.0 1.0 1.0
- link head_pan_link: mass 6.339 -> None; geometry collision mesh filename=package://pycram/resources/pr2/stl/head_pan_L.stl scale=1.0 1.0 1.0
- link head_plate_frame: mass 0.01 -> None; geometry collision box size=0.01 0.01 0.01
- link head_tilt_link: mass 4.479 -> None; geometry collision mesh filename=package://pycram/resources/pr2/stl/head_tilt_L.stl scale=1.0 1.0 1.0
- link high_def_frame: mass 0.01 -> None
- link high_def_optical_frame: mass 0.01 -> None
- link imu_link: mass 0.001 -> None
- link l_elbow_flex_link: mass 1.90327 -> None; geometry collision mesh filename=package://pycram/resources/pr2/stl/elbow_flex.stl scale=1.0 1.0 1.0
- link l_forearm_cam_frame: mass 0.01 -> None
- link l_forearm_link: mass 2.57968 -> None; geometry collision mesh filename=package://pycram/resources/pr2/stl/forearm.stl scale=1.0 1.0 1.0
- link l_forearm_roll_link: mass 0.1 -> None; geometry collision mesh filename=package://pycram/resources/pr2/stl/forearm_roll_L.stl scale=1.0 1.0 1.0
- link l_gripper_l_finger_link: mass 0.17126 -> None; geometry collision mesh filename=package://pycram/resources/pr2/stl/l_finger.stl scale=1.0 1.0 1.0
- link l_gripper_l_finger_tip_link: mass 0.04419 -> None; geometry collision mesh filename=package://pycram/resources/pr2/stl/l_finger_tip.stl scale=1.0 1.0 1.0
- link l_gripper_motor_accelerometer_link: mass 0.001 -> None; geometry collision box size=0.001 0.001 0.001
- link l_gripper_motor_screw_link: mass 0.01 -> None
- link l_gripper_motor_slider_link: mass 0.01 -> None
- link l_gripper_palm_link: mass 0.58007 -> None; geometry collision mesh filename=package://pycram/resources/pr2/stl/gripper_palm.stl scale=1.0 1.0 1.0
- link l_gripper_r_finger_link: mass 0.17389 -> None; geometry collision mesh filename=package://pycram/resources/pr2/stl/l_finger.stl scale=1.0 1.0 1.0
- link l_gripper_r_finger_tip_link: mass 0.04419 -> None; geometry collision mesh filename=package://pycram/resources/pr2/stl/l_finger_tip.stl scale=1.0 1.0 1.0
- link l_shoulder_lift_link: mass 2.74988 -> None; geometry collision mesh filename=package://pycram/resources/pr2/stl/shoulder_lift.stl scale=1.0 1.0 1.0
- link l_shoulder_pan_link: mass 25.799322 -> None; geometry collision mesh filename=package://pycram/resources/pr2/stl/shoulder_pan.stl scale=1.0 1.0 1.0
- link l_torso_lift_side_plate_link: mass 0.1 -> None
- link l_upper_arm_link: mass 6.01769 -> None; geometry collision mesh filename=package://pycram/resources/pr2/stl/upper_arm.stl scale=1.0 1.0 1.0
- link l_upper_arm_roll_link: mass 0.1 -> None; geometry collision mesh filename=package://pycram/resources/pr2/stl/upper_arm_roll_L.stl scale=1.0 1.0 1.0
- link l_wrist_flex_link: mass 0.61402 -> None; geometry collision mesh filename=package://pycram/resources/pr2/stl/wrist_flex.stl scale=1.0 1.0 1.0
- link l_wrist_roll_link: mass 0.1 -> None; geometry collision mesh filename=package://pycram/resources/pr2/stl/wrist_roll_L.stl scale=1.0 1.0 1.0
- link laser_tilt_link: mass 0.001 -> None
- link laser_tilt_mount_link: mass 0.591 -> None; geometry collision mesh filename=package://pycram/resources/pr2/stl/tilting_hokuyo_L.stl scale=1.0 1.0 1.0
- link narrow_stereo_l_stereo_camera_frame: mass 0.01 -> None
- link narrow_stereo_link: mass 0.1 -> None
- link narrow_stereo_r_stereo_camera_frame: mass 0.01 -> None
- link projector_wg6802418_child_frame: mass 0.01 -> None
- link projector_wg6802418_frame: mass 0.01 -> None
- link r_elbow_flex_link: mass 1.90327 -> None; geometry collision mesh filename=package://pycram/resources/pr2/stl/elbow_flex.stl scale=1.0 1.0 1.0
- link r_forearm_cam_frame: mass 0.01 -> None
- link r_forearm_link: mass 2.57968 -> None; geometry collision mesh filename=package://pycram/resources/pr2/stl/forearm.stl scale=1.0 1.0 1.0
- link r_forearm_roll_link: mass 0.1 -> None; geometry collision mesh filename=package://pycram/resources/pr2/stl/forearm_roll_L.stl scale=1.0 1.0 1.0
- link r_gripper_l_finger_link: mass 0.17126 -> None; geometry collision mesh filename=package://pycram/resources/pr2/stl/l_finger.stl scale=1.0 1.0 1.0
- link r_gripper_l_finger_tip_link: mass 0.04419 -> None; geometry collision mesh filename=package://pycram/resources/pr2/stl/l_finger_tip.stl scale=1.0 1.0 1.0
- link r_gripper_motor_accelerometer_link: mass 0.001 -> None; geometry collision box size=0.001 0.001 0.001
- link r_gripper_motor_screw_link: mass 0.01 -> None
- link r_gripper_motor_slider_link: mass 0.01 -> None
- link r_gripper_palm_link: mass 0.58007 -> None; geometry collision mesh filename=package://pycram/resources/pr2/stl/gripper_palm.stl scale=1.0 1.0 1.0
- link r_gripper_r_finger_link: mass 0.17389 -> None; geometry collision mesh filename=package://pycram/resources/pr2/stl/l_finger.stl scale=1.0 1.0 1.0
- link r_gripper_r_finger_tip_link: mass 0.04419 -> None; geometry collision mesh filename=package://pycram/resources/pr2/stl/l_finger_tip.stl scale=1.0 1.0 1.0
- link r_shoulder_lift_link: mass 2.74988 -> None; geometry collision mesh filename=package://pycram/resources/pr2/stl/shoulder_lift.stl scale=1.0 1.0 1.0
- link r_shoulder_pan_link: mass 25.799322 -> None; geometry collision mesh filename=package://pycram/resources/pr2/stl/shoulder_pan.stl scale=1.0 1.0 1.0
- link r_torso_lift_side_plate_link: mass 0.1 -> None
- link r_upper_arm_link: mass 6.01769 -> None; geometry collision mesh filename=package://pycram/resources/pr2/stl/upper_arm.stl scale=1.0 1.0 1.0
- link r_upper_arm_roll_link: mass 0.1 -> None; geometry collision mesh filename=package://pycram/resources/pr2/stl/upper_arm_roll_L.stl scale=1.0 1.0 1.0
- link r_wrist_flex_link: mass 0.61402 -> None; geometry collision mesh filename=package://pycram/resources/pr2/stl/wrist_flex.stl scale=1.0 1.0 1.0
- link r_wrist_roll_link: mass 0.1 -> None; geometry collision mesh filename=package://pycram/resources/pr2/stl/wrist_roll_L.stl scale=1.0 1.0 1.0
- link sensor_mount_link: mass 0.05 -> None; geometry 
- link torso_lift_link: mass 36.248046 -> None; geometry collision mesh filename=package://pycram/resources/pr2/stl/torso_lift_L.stl scale=1.0 1.0 1.0
- link torso_lift_motor_screw_link: mass 1.0 -> None
- link wide_stereo_l_stereo_camera_frame: mass 0.01 -> None
- link wide_stereo_link: mass 0.1 -> None
- link wide_stereo_optical_frame: mass 0.1 -> None
- link wide_stereo_r_stereo_camera_frame: mass 0.01 -> None
Joints:
- removed joint base_bellow_joint
- removed joint base_footprint_joint
- removed joint base_laser_joint
- removed joint double_stereo_frame_joint
- removed joint imu_joint
- removed joint l_forearm_joint
- removed joint l_gripper_led_joint
- removed joint l_gripper_motor_accelerometer_joint
- removed joint l_gripper_palm_joint
- removed joint l_gripper_tool_joint
- removed joint l_torso_lift_side_plate_joint
- removed joint l_upper_arm_joint
- removed joint laser_tilt_joint
- removed joint narrow_stereo_frame_joint
- removed joint r_forearm_joint
- removed joint r_gripper_led_joint
- removed joint r_gripper_motor_accelerometer_joint
- removed joint r_gripper_palm_joint
- removed joint r_gripper_tool_joint
- removed joint r_torso_lift_side_plate_joint
- removed joint r_upper_arm_joint
- removed joint sensor_mount_frame_joint
- removed joint wide_stereo_frame_joint
- added joint base_bellow_link_joint: type fixed, parent base_link, child base_bellow_link, origin xyz=-0.29 0.0 0.8 rpy=0.0 -0.0 0.0
- added joint base_laser_link_joint: type fixed, parent base_link, child base_laser_link, origin xyz=0.275 0.0 0.252 rpy=0.0 -0.0 0.0
- added joint base_link_joint: type fixed, parent base_footprint, child base_link, origin xyz=0.0 0.0 0.051 rpy=0.0 -0.0 0.0
- added joint double_stereo_link_joint: type fixed, parent sensor_mount_link, child double_stereo_link, origin xyz=0.0 0.0 0.0 rpy=0.0 -0.0 0.0
- added joint imu_link_joint: type fixed, parent torso_lift_link, child imu_link, origin xyz=-0.02977 -0.1497 0.164 rpy=3.141592653589793 -2.0682310711021437e-13 3.141592653589793
- added joint l_forearm_link_joint: type fixed, parent l_forearm_roll_link, child l_forearm_link, origin xyz=0.0 0.0 0.0 rpy=0.0 -0.0 0.0
- added joint l_gripper_led_frame_joint: type fixed, parent l_gripper_palm_link, child l_gripper_led_frame, origin xyz=0.0513 0.0 0.0244 rpy=0.0 -0.0 0.0
- added joint l_gripper_motor_accelerometer_link_joint: type fixed, parent l_gripper_palm_link, child l_gripper_motor_accelerometer_link, origin xyz=0.0 0.0 0.0 rpy=0.0 -0.0 0.0
- added joint l_gripper_palm_link_joint: type fixed, parent l_wrist_roll_link, child l_gripper_palm_link, origin xyz=0.0 0.0 0.0 rpy=0.0 -0.0 0.0
- added joint l_gripper_tool_frame_joint: type fixed, parent l_gripper_palm_link, child l_gripper_tool_frame, origin xyz=0.18 0.0 0.0 rpy=0.0 -0.0 0.0
- added joint l_torso_lift_side_plate_link_joint: type fixed, parent torso_lift_link, child l_torso_lift_side_plate_link, origin xyz=0.0535 0.209285 0.176625 rpy=0.0 -0.0 0.0
- added joint l_upper_arm_link_joint: type fixed, parent l_upper_arm_roll_link, child l_upper_arm_link, origin xyz=0.0 0.0 0.0 rpy=0.0 -0.0 0.0
- added joint laser_tilt_link_joint: type fixed, parent laser_tilt_mount_link, child laser_tilt_link, origin xyz=0.0 0.0 0.03 rpy=0.0 -0.0 0.0
- added joint narrow_stereo_link_joint: type fixed, parent double_stereo_link, child narrow_stereo_link, origin xyz=0.045 0.06 0.0501 rpy=0.0 -0.0 0.0
- added joint r_forearm_link_joint: type fixed, parent r_forearm_roll_link, child r_forearm_link, origin xyz=0.0 0.0 0.0 rpy=0.0 -0.0 0.0
- added joint r_gripper_led_frame_joint: type fixed, parent r_gripper_palm_link, child r_gripper_led_frame, origin xyz=0.0513 0.0 0.0244 rpy=0.0 -0.0 0.0
- added joint r_gripper_motor_accelerometer_link_joint: type fixed, parent r_gripper_palm_link, child r_gripper_motor_accelerometer_link, origin xyz=0.0 0.0 0.0 rpy=0.0 -0.0 0.0
- added joint r_gripper_palm_link_joint: type fixed, parent r_wrist_roll_link, child r_gripper_palm_link, origin xyz=0.0 0.0 0.0 rpy=0.0 -0.0 0.0
- added joint r_gripper_tool_frame_joint: type fixed, parent r_gripper_palm_link, child r_gripper_tool_frame, origin xyz=0.18 0.0 0.0 rpy=0.0 -0.0 0.0
- added joint r_torso_lift_side_plate_link_joint: type fixed, parent torso_lift_link, child r_torso_lift_side_plate_link, origin xyz=0.0535 -0.209285 0.176625 rpy=0.0 -0.0 0.0
- added joint r_upper_arm_link_joint: type fixed, parent r_upper_arm_roll_link, child r_upper_arm_link, origin xyz=0.0 0.0 0.0 rpy=0.0 -0.0 0.0
- added joint sensor_mount_link_joint: type fixed, parent head_plate_frame, child sensor_mount_link, origin xyz=0.0 0.0 0.0 rpy=0.0 -0.0 0.0
- added joint wide_stereo_link_joint: type fixed, parent double_stereo_link, child wide_stereo_link, origin xyz=0.045 0.03 0.0501 rpy=0.0 -0.0 0.0
- joint bl_caster_l_wheel_joint: limit effort=7 velocity=15 -> (none); origin xyz=0 0.049 0 rpy=0 0 0 -> xyz=0.0 0.04899999871850014 0.0 rpy=0.0 -0.0 0.0
- joint bl_caster_r_wheel_joint: limit effort=7 velocity=15 -> (none); origin xyz=0 -0.049 0 rpy=0 0 0 -> xyz=0.0 -0.04899999871850014 0.0 rpy=0.0 -0.0 0.0
- joint bl_caster_rotation_joint: limit effort=6.5 velocity=10 -> (none); origin xyz=-0.2246 0.2246 0.0282 rpy=0 0 0 -> xyz=-0.22460000216960907 0.22460000216960907 0.028200000524520874 rpy=0.0 -0.0 0.0
- joint br_caster_l_wheel_joint: limit effort=7 velocity=15 -> (none); origin xyz=0 0.049 0 rpy=0 0 0 -> xyz=0.0 0.04899999871850014 0.0 rpy=0.0 -0.0 0.0
- joint br_caster_r_wheel_joint: limit effort=7 velocity=15 -> (none); origin xyz=0 -0.049 0 rpy=0 0 0 -> xyz=0.0 -0.04899999871850014 0.0 rpy=0.0 -0.0 0.0
- joint br_caster_rotation_joint: limit effort=6.5 velocity=10 -> (none); origin xyz=-0.2246 -0.2246 0.0282 rpy=0 0 0 -> xyz=-0.22460000216960907 -0.22460000216960907 0.028200000524520874 rpy=0.0 -0.0 0.0
- joint fl_caster_l_wheel_joint: limit effort=7 velocity=15 -> (none); origin xyz=0 0.049 0 rpy=0 0 0 -> xyz=0.0 0.04899999871850014 0.0 rpy=0.0 -0.0 0.0
- joint fl_caster_r_wheel_joint: limit effort=7 velocity=15 -> (none); origin xyz=0 -0.049 0 rpy=0 0 0 -> xyz=0.0 -0.04899999871850014 0.0 rpy=0.0 -0.0 0.0
- joint fl_caster_rotation_joint: limit effort=6.5 velocity=10 -> (none); origin xyz=0.2246 0.2246 0.0282 rpy=0 0 0 -> xyz=0.22460000216960907 0.22460000216960907 0.028200000524520874 rpy=0.0 -0.0 0.0
- joint fr_caster_l_wheel_joint: limit effort=7 velocity=15 -> (none); origin xyz=0 0.049 0 rpy=0 0 0 -> xyz=0.0 0.04899999871850014 0.0 rpy=0.0 -0.0 0.0
- joint fr_caster_r_wheel_joint: limit effort=7 velocity=15 -> (none); origin xyz=0 -0.049 0 rpy=0 0 0 -> xyz=0.0 -0.04899999871850014 0.0 rpy=0.0 -0.0 0.0
- joint fr_caster_rotation_joint: limit effort=6.5 velocity=10 -> (none); origin xyz=0.2246 -0.2246 0.0282 rpy=0 0 0 -> xyz=0.22460000216960907 -0.22460000216960907 0.028200000524520874 rpy=0.0 -0.0 0.0
- joint head_pan_joint: limit lower=-3.007 upper=3.007 effort=2.645 velocity=6 -> lower=-3.0069999542066057 upper=3.0069999542066057 effort=1000 velocity=1000; origin xyz=-0.01707 0.0 0.38145 rpy=0.0 0.0 0.0 -> xyz=-0.017069999128580093 0.0 0.38144999742507935 rpy=0.0 -0.0 0.0
- joint head_plate_frame_joint: origin xyz=0.0232 0 0.0645 rpy=0 0 0 -> xyz=0.0232 0.0 0.0645 rpy=0.0 -0.0 0.0
- joint head_tilt_joint: limit lower=-0.471238 upper=1.39626 effort=18 velocity=5 -> lower=-0.4712379992216011 upper=1.3962599394860464 effort=1000 velocity=1000; origin xyz=0.068 0 0 rpy=0 0 0 -> xyz=0.06800000369548798 0.0 0.0 rpy=0.0 -0.0 0.0
- joint high_def_frame_joint: origin xyz=0.046457 -0.110 0.054600 rpy=0 0 0 -> xyz=0.046457 -0.11 0.0546 rpy=0.0 -0.0 0.0
- joint high_def_optical_frame_joint: origin xyz=0.0            0.0         0.0 rpy=-1.57079632679 0.0 -1.57079632679 -> xyz=0.0 0.0 0.0 rpy=-1.5707963267900003 -0.0 -1.5707963267900003
- joint l_elbow_flex_joint: limit lower=-2.3213 upper=0.00 effort=30 velocity=3.3 -> lower=-2.3212998893773635 upper=0.0 effort=1000 velocity=1000; origin xyz=0.4 0 0 rpy=0 0 0 -> xyz=0.4000000059604645 0.0 0.0 rpy=0.0 -0.0 0.0
- joint l_forearm_cam_frame_joint: origin xyz=.135 0 .044 rpy=-1.57079632679 -0.562868683768 0 -> xyz=0.135 0.0 0.044 rpy=-1.570796326789999 -0.5628686837679997 -1.9691140508801486e-16
- joint l_forearm_cam_optical_frame_joint: origin xyz=0 0 0 rpy=-1.57079632679 0.0 -1.57079632679 -> xyz=0.0 0.0 0.0 rpy=-1.5707963267900003 -0.0 -1.5707963267900003
- joint l_forearm_roll_joint: limit effort=30 velocity=3.6 -> (none); origin xyz=0 0 0 rpy=0 0 0 -> xyz=0.0 0.0 0.0 rpy=0.0 -0.0 0.0
- joint l_gripper_joint: limit lower=0.0 upper=0.09 effort=1000.0 velocity=0.2 -> lower=0.0 upper=0.09000000357627869 effort=1000 velocity=1000; origin (none) -> xyz=0.0 0.0 0.0 rpy=0.0 -0.0 0.0
- joint l_gripper_l_finger_joint: limit lower=0.0 upper=0.548 effort=1000.0 velocity=0.5 -> lower=0.0 upper=0.5479999890861499 effort=1000 velocity=1000; origin xyz=0.07691 0.01 0 rpy=0 0 0 -> xyz=0.07690999656915665 0.009999999776482582 0.0 rpy=0.0 -0.0 0.0
- joint l_gripper_l_finger_tip_joint: limit lower=0.0 upper=0.548 effort=1000.0 velocity=0.5 -> lower=0.0 upper=0.5479999890861499 effort=1000 velocity=1000; origin xyz=0.09137 0.00495 0 rpy=0 0 0 -> xyz=0.09137000143527985 0.00494999997317791 0.0 rpy=0.0 -0.0 0.0
- joint l_gripper_motor_screw_joint: origin xyz=0.0 0 0 rpy=0 0 0 -> xyz=0.0 0.0 0.0 rpy=0.0 -0.0 0.0
- joint l_gripper_motor_slider_joint: limit lower=-0.1 upper=0.1 effort=1000.0 velocity=0.2 -> lower=-0.10000000149011612 upper=0.10000000149011612 effort=1000 velocity=1000; origin xyz=0.16828 0 0 rpy=0 0 0 -> xyz=0.1682800054550171 0.0 0.0 rpy=0.0 -0.0 0.0
- joint l_gripper_r_finger_joint: limit lower=0.0 upper=0.548 effort=1000.0 velocity=0.5 -> lower=0.0 upper=0.5479999890861499 effort=1000 velocity=1000; origin xyz=0.07691 -0.01 0 rpy=0 0 0 -> xyz=0.07690999656915665 -0.009999999776482582 0.0 rpy=0.0 -0.0 0.0
- joint l_gripper_r_finger_tip_joint: limit lower=0.0 upper=0.548 effort=1000.0 velocity=0.5 -> lower=0.0 upper=0.5479999890861499 effort=1000 velocity=1000; origin xyz=0.09137 -0.00495 0 rpy=0 0 0 -> xyz=0.09137000143527985 -0.00494999997317791 0.0 rpy=0.0 -0.0 0.0
- joint l_shoulder_lift_joint: limit lower=-0.5236 upper=1.3963 effort=30 velocity=2.082 -> lower=-0.523600007310303 upper=1.3963000200604523 effort=1000 velocity=1000; origin xyz=0.1 0 0 rpy=0 0 0 -> xyz=0.10000000149011612 0.0 0.0 rpy=0.0 -0.0 0.0
- joint l_shoulder_pan_joint: limit lower=-0.714601836603 upper=2.2853981634 effort=30 velocity=2.088 -> lower=-0.7146018208222451 upper=2.2853980810381143 effort=1000 velocity=1000; origin xyz=0.0 0.188 0.0 rpy=0 0 0 -> xyz=0.0 0.18799999356269836 0.0 rpy=0.0 -0.0 0.0
- joint l_upper_arm_roll_joint: limit lower=-0.8 upper=3.9 effort=30 velocity=3.27 -> lower=-0.8000000093382438 upper=3.8999999456553973 effort=1000 velocity=1000; origin xyz=0 0 0 rpy=0 0 0 -> xyz=0.0 0.0 0.0 rpy=0.0 -0.0 0.0
- joint l_wrist_flex_joint: limit lower=-2.18 upper=0.0 effort=10 velocity=3.078 -> lower=-2.1800000187888116 upper=0.0 effort=1000 velocity=1000; origin xyz=0.321 0 0 rpy=0 0 0 -> xyz=0.32100000977516174 0.0 0.0 rpy=0.0 -0.0 0.0
- joint l_wrist_roll_joint: limit effort=10 velocity=3.6 -> (none); origin xyz=0 0 0 rpy=0 0 0 -> xyz=0.0 0.0 0.0 rpy=0.0 -0.0 0.0
- joint laser_tilt_mount_joint: limit lower=-0.7854 upper=1.48353 effort=0.65 velocity=10.0 -> lower=-0.7854000276102113 upper=1.4835299973532345 effort=1000 velocity=1000; origin xyz=0.09893 0 0.227 rpy=0 0 0 -> xyz=0.0989300012588501 0.0 0.22699999809265137 rpy=0.0 -0.0 0.0
- joint narrow_stereo_l_stereo_camera_frame_joint: origin xyz=0 0 0 rpy=0 0 0 -> xyz=0.0 0.0 0.0 rpy=0.0 -0.0 0.0
- joint narrow_stereo_l_stereo_camera_optical_frame_joint: origin xyz=0 0 0 rpy=-1.57079632679 0.0 -1.57079632679 -> xyz=0.0 0.0 0.0 rpy=-1.5707963267900003 -0.0 -1.5707963267900003
- joint narrow_stereo_optical_frame_joint: origin xyz=0 0 0 rpy=-1.57079632679 0.0 -1.57079632679 -> xyz=0.0 0.0 0.0 rpy=-1.5707963267900003 -0.0 -1.5707963267900003
- joint narrow_stereo_r_stereo_camera_frame_joint: origin xyz=0.0 -0.09 0.0 rpy=0.0 0.0 0.0 -> xyz=0.0 -0.09 0.0 rpy=0.0 -0.0 0.0
- joint narrow_stereo_r_stereo_camera_optical_frame_joint: origin xyz=0 0 0 rpy=-1.57079632679 0.0 -1.57079632679 -> xyz=0.0 0.0 0.0 rpy=-1.5707963267900003 -0.0 -1.5707963267900003
- joint projector_wg6802418_child_frame_joint: origin xyz=0 0 0 rpy=0 -1.57079632679 0 -> xyz=0.0 0.0 0.0 rpy=0.0 -1.57079632679 0.0
- joint projector_wg6802418_frame_joint: origin xyz=0 0.110 0.0546 rpy=0 0 0 -> xyz=0.0 0.11 0.0546 rpy=0.0 -0.0 0.0
- joint r_elbow_flex_joint: limit lower=-2.3213 upper=0.00 effort=30 velocity=3.3 -> lower=-2.3212998893773635 upper=0.0 effort=1000 velocity=1000; origin xyz=0.4 0 0 rpy=0 0 0 -> xyz=0.4000000059604645 0.0 0.0 rpy=0.0 -0.0 0.0
- joint r_forearm_cam_frame_joint: origin xyz=.135 0 .044 rpy=1.57079632679 -0.562868683768 0 -> xyz=0.135 0.0 0.044 rpy=1.570796326789999 -0.5628686837679997 1.9691140508801486e-16
- joint r_forearm_cam_optical_frame_joint: origin xyz=0 0 0 rpy=-1.57079632679 0.0 -1.57079632679 -> xyz=0.0 0.0 0.0 rpy=-1.5707963267900003 -0.0 -1.5707963267900003
- joint r_forearm_roll_joint: limit effort=30 velocity=3.6 -> (none); origin xyz=0 0 0 rpy=0 0 0 -> xyz=0.0 0.0 0.0 rpy=0.0 -0.0 0.0
- joint r_gripper_joint: limit lower=0.0 upper=0.09 effort=1000.0 velocity=0.2 -> lower=0.0 upper=0.09000000357627869 effort=1000 velocity=1000; origin (none) -> xyz=0.0 0.0 0.0 rpy=0.0 -0.0 0.0
- joint r_gripper_l_finger_joint: limit lower=0.0 upper=0.548 effort=1000.0 velocity=0.5 -> lower=0.0 upper=0.5479999890861499 effort=1000 velocity=1000; origin xyz=0.07691 0.01 0 rpy=0 0 0 -> xyz=0.07690999656915665 0.009999999776482582 0.0 rpy=0.0 -0.0 0.0
- joint r_gripper_l_finger_tip_joint: limit lower=0.0 upper=0.548 effort=1000.0 velocity=0.5 -> lower=0.0 upper=0.5479999890861499 effort=1000 velocity=1000; origin xyz=0.09137 0.00495 0 rpy=0 0 0 -> xyz=0.09137000143527985 0.00494999997317791 0.0 rpy=0.0 -0.0 0.0
- joint r_gripper_motor_screw_joint: origin xyz=0.0 0 0 rpy=0 0 0 -> xyz=0.0 0.0 0.0 rpy=0.0 -0.0 0.0
- joint r_gripper_motor_slider_joint: limit lower=-0.1 upper=0.1 effort=1000.0 velocity=0.2 -> lower=-0.10000000149011612 upper=0.10000000149011612 effort=1000 velocity=1000; origin xyz=0.16828 0 0 rpy=0 0 0 -> xyz=0.1682800054550171 0.0 0.0 rpy=0.0 -0.0 0.0
- joint r_gripper_r_finger_joint: limit lower=0.0 upper=0.548 effort=1000.0 velocity=0.5 -> lower=0.0 upper=0.5479999890861499 effort=1000 velocity=1000; origin xyz=0.07691 -0.01 0 rpy=0 0 0 -> xyz=0.07690999656915665 -0.009999999776482582 0.0 rpy=0.0 -0.0 0.0
- joint r_gripper_r_finger_tip_joint: limit lower=0.0 upper=0.548 effort=1000.0 velocity=0.5 -> lower=0.0 upper=0.5479999890861499 effort=1000 velocity=1000; origin xyz=0.09137 -0.00495 0 rpy=0 0 0 -> xyz=0.09137000143527985 -0.00494999997317791 0.0 rpy=0.0 -0.0 0.0
- joint r_shoulder_lift_joint: limit lower=-0.5236 upper=1.3963 effort=30 velocity=2.082 -> lower=-0.523600007310303 upper=1.3963000200604523 effort=1000 velocity=1000; origin xyz=0.1 0 0 rpy=0 0 0 -> xyz=0.10000000149011612 0.0 0.0 rpy=0.0 -0.0 0.0
- joint r_shoulder_pan_joint: limit lower=-2.2853981634 upper=0.714601836603 effort=30 velocity=2.088 -> lower=-2.2853980810381143 upper=0.7146018208222451 effort=1000 velocity=1000; origin xyz=0.0 -0.188 0.0 rpy=0 0 0 -> xyz=0.0 -0.18799999356269836 0.0 rpy=0.0 -0.0 0.0
- joint r_upper_arm_roll_joint: limit lower=-3.9 upper=0.8 effort=30 velocity=3.27 -> lower=-3.8999999456553973 upper=0.8000000093382438 effort=1000 velocity=1000; origin xyz=0 0 0 rpy=0 0 0 -> xyz=0.0 0.0 0.0 rpy=0.0 -0.0 0.0
- joint r_wrist_flex_joint: limit lower=-2.18 upper=0.0 effort=10 velocity=3.078 -> lower=-2.1800000187888116 upper=0.0 effort=1000 velocity=1000; origin xyz=0.321 0 0 rpy=0 0 0 -> xyz=0.32100000977516174 0.0 0.0 rpy=0.0 -0.0 0.0
- joint r_wrist_roll_joint: limit effort=10 velocity=3.6 -> (none); origin xyz=0 0 0 rpy=0 0 0 -> xyz=0.0 0.0 0.0 rpy=0.0 -0.0 0.0
- joint torso_lift_joint: limit lower=0. upper=0.33 effort=1000 velocity=0.13 -> lower=0.0 upper=0.33000001311302185 effort=1000 velocity=1000; origin xyz=-0.05 0 0.739675 rpy=0 0 0 -> xyz=-0.05000000074505806 0.0 0.739674985408783 rpy=0.0 -0.0 0.0
- joint torso_lift_motor_screw_joint: origin xyz=-0.15 0.0 0.7 -> xyz=-0.15000000596046448 0.0 0.699999988079071 rpy=0.0 -0.0 0.0
- joint wide_stereo_l_stereo_camera_frame_joint: origin xyz=0 0 0 rpy=0 0 0 -> xyz=0.0 0.0 0.0 rpy=0.0 -0.0 0.0
- joint wide_stereo_l_stereo_camera_optical_frame_joint: origin xyz=0 0 0 rpy=-1.57079632679 0.0 -1.57079632679 -> xyz=0.0 0.0 0.0 rpy=-1.5707963267900003 -0.0 -1.5707963267900003
- joint wide_stereo_optical_frame_joint: origin xyz=0 0 0 rpy=-1.57079632679 0.0 -1.57079632679 -> xyz=0.0 0.0 0.0 rpy=-1.5707963267900003 -0.0 -1.5707963267900003
- joint wide_stereo_r_stereo_camera_frame_joint: origin xyz=0.0 -0.09 0.0 rpy=0.0 0.0 0.0 -> xyz=0.0 -0.09 0.0 rpy=0.0 -0.0 0.0
- joint wide_stereo_r_stereo_camera_optical_frame_joint: origin xyz=0 0 0 rpy=-1.57079632679 0.0 -1.57079632679 -> xyz=0.0 0.0 0.0 rpy=-1.5707963267900003 -0.0 -1.5707963267900003
