Commit message: [resources]: reverted pr2 and kitchen. removed mor unused files

File: resources/worlds/kitchen.urdf (robot description, URDF)
Before this commit: robot iai_oven_area, 85 links, 84 joints
Links:
- removed link second_table_area
Joints:
- removed joint second_table_area_joint
- joint table_area_main_joint: origin xyz=-2.7 2.55 0 rpy=0 0 3.14159265359 -> xyz=-1.4 -1.05 0 rpy=0 0 3.14159265359
