Commit message: Black fuck up

File: resources/worlds/apartment.urdf (robot description, URDF)
Before this commit: robot apartment, 113 links, 112 joints
Links:
- link walls: geometry collision mesh filename=package://iai_apartment/meshes/collision/walls.stl; visual mesh filename=package://iai_apartment/meshes/visual/walls.dae

Commit message: Fixed Probability semantic costmap

File: resources/worlds/apartment.urdf (robot description, URDF)
Before this commit: robot apartment, 113 links, 112 joints
Links:
- link walls: geometry collision box size=1 1 1; visual mesh filename=package://iai_apartment/meshes/visual/walls.dae
