Commit message: [justin] swapped out stl files with dae files

File: resources/robots/rollin_justin.urdf (robot description, URDF)
Before this commit: robot rollin_justin, 66 links, 65 joints
Links:
- link base_link: geometry collision mesh filename=package://iai_dlr_rollin_justin/mjcf/rollin-justin/meshes/d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 scale=1 1 1; visual mesh filename=package://iai_dlr_rollin_justin/mjcf/rollin-justin/meshes/d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 scale=1 1 1
- link head1: geometry collision mesh filename=package://iai_dlr_rollin_justin/mjcf/rollin-justin/meshes/d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 scale=1 1 1; visual mesh filename=package://iai_dlr_rollin_justin/mjcf/rollin-justin/meshes/d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 scale=1 1 1
- link head2: geometry collision mesh filename=package://iai_dlr_rollin_justin/mjcf/rollin-justin/meshes/d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 scale=1 1 1; visual mesh filename=package://iai_dlr_rollin_justin/mjcf/rollin-justin/meshes/d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 scale=1 1 1
- link left_1thumb2: geometry collision mesh filename=package://iai_dlr_rollin_justin/mjcf/rollin-justin/meshes/d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 scale=1 1 1; visual mesh filename=package://iai_dlr_rollin_justin/mjcf/rollin-justin/meshes/d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 scale=1 1 1
- link left_1thumb3: geometry collision mesh filename=package://iai_dlr_rollin_justin/mjcf/rollin-justin/meshes/d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 scale=1 1 1; visual mesh filename=package://iai_dlr_rollin_justin/mjcf/rollin-justin/meshes/d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 scale=1 1 1
- link left_1thumb4: geometry collision mesh filename=package://iai_dlr_rollin_justin/mjcf/rollin-justin/meshes/d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 scale=1 1 1; visual mesh filename=package://iai_dlr_rollin_justin/mjcf/rollin-justin/meshes/d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 scale=1 1 1
- link left_1thumb_base: geometry visual mesh filename=package://iai_dlr_rollin_justin/mjcf/rollin-justin/meshes/d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 scale=1 1 1
- link left_2tip2: geometry collision mesh filename=package://iai_dlr_rollin_justin/mjcf/rollin-justin/meshes/d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 scale=1 1 1; visual mesh filename=package://iai_dlr_rollin_justin/mjcf/rollin-justin/meshes/d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 scale=1 1 1
- link left_2tip3: geometry collision mesh filename=package://iai_dlr_rollin_justin/mjcf/rollin-justin/meshes/d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 scale=1 1 1; visual mesh filename=package://iai_dlr_rollin_justin/mjcf/rollin-justin/meshes/d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 scale=1 1 1
- link left_2tip4: geometry collision mesh filename=package://iai_dlr_rollin_justin/mjcf/rollin-justin/meshes/d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 scale=1 1 1; visual mesh filename=package://iai_dlr_rollin_justin/mjcf/rollin-justin/meshes/d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 scale=1 1 1
- link left_2tip_base: geometry visual mesh filename=package://iai_dlr_rollin_justin/mjcf/rollin-justin/meshes/d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 scale=1 1 1
- link left_3middle2: geometry collision mesh filename=package://iai_dlr_rollin_justin/mjcf/rollin-justin/meshes/d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 scale=1 1 1; visual mesh filename=package://iai_dlr_rollin_justin/mjcf/rollin-justin/meshes/d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 scale=1 1 1
- link left_3middle3: geometry collision mesh filename=package://iai_dlr_rollin_justin/mjcf/rollin-justin/meshes/d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 scale=1 1 1; visual mesh filename=package://iai_dlr_rollin_justin/mjcf/rollin-justin/meshes/d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 scale=1 1 1
- link left_3middle4: geometry collision mesh filename=package://iai_dlr_rollin_justin/mjcf/rollin-justin/meshes/d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 scale=1 1 1; visual mesh filename=package://iai_dlr_rollin_justin/mjcf/rollin-justin/meshes/d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 scale=1 1 1
- link left_3middle_base: geometry collision mesh filename=package://iai_dlr_rollin_justin/mjcf/rollin-justin/meshes/d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 scale=1 1 1; visual mesh filename=package://iai_dlr_rollin_justin/mjcf/rollin-justin/meshes/d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 scale=1 1 1
- link left_4ring2: geometry collision mesh filename=package://iai_dlr_rollin_justin/mjcf/rollin-justin/meshes/d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 scale=1 1 1; visual mesh filename=package://iai_dlr_rollin_justin/mjcf/rollin-justin/meshes/d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 scale=1 1 1
- link left_4ring3: geometry collision mesh filename=package://iai_dlr_rollin_justin/mjcf/rollin-justin/meshes/d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 scale=1 1 1; visual mesh filename=package://iai_dlr_rollin_justin/mjcf/rollin-justin/meshes/d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 scale=1 1 1
- link left_4ring4: geometry collision mesh filename=package://iai_dlr_rollin_justin/mjcf/rollin-justin/meshes/d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 scale=1 1 1; visual mesh filename=package://iai_dlr_rollin_justin/mjcf/rollin-justin/meshes/d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 scale=1 1 1
- link left_4ring_base: geometry visual mesh filename=package://iai_dlr_rollin_justin/mjcf/rollin-justin/meshes/d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 scale=1 1 1
- link left_arm1: geometry collision mesh filename=package://iai_dlr_rollin_justin/mjcf/rollin-justin/meshes/d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 scale=1 1 1; visual mesh filename=package://iai_dlr_rollin_justin/mjcf/rollin-justin/meshes/d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 scale=1 1 1
- link left_arm2: geometry collision mesh filename=package://iai_dlr_rollin_justin/mjcf/rollin-justin/meshes/d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 scale=1 1 1; visual mesh filename=package://iai_dlr_rollin_justin/mjcf/rollin-justin/meshes/d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 scale=1 1 1
- link left_arm3: geometry collision mesh filename=package://iai_dlr_rollin_justin/mjcf/rollin-justin/meshes/d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 scale=1 1 1; visual mesh filename=package://iai_dlr_rollin_justin/mjcf/rollin-justin/meshes/d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 scale=1 1 1
- link left_arm4: geometry collision mesh filename=package://iai_dlr_rollin_justin/mjcf/rollin-justin/meshes/d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 scale=1 1 1; visual mesh filename=package://iai_dlr_rollin_justin/mjcf/rollin-justin/meshes/d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 scale=1 1 1
- link left_arm5: geometry collision mesh filename=package://iai_dlr_rollin_justin/mjcf/rollin-justin/meshes/d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 scale=1 1 1; visual mesh filename=package://iai_dlr_rollin_justin/mjcf/rollin-justin/meshes/d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 scale=1 1 1
- link left_arm6: geometry collision mesh filename=package://iai_dlr_rollin_justin/mjcf/rollin-justin/meshes/d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 scale=1 1 1; visual mesh filename=package://iai_dlr_rollin_justin/mjcf/rollin-justin/meshes/d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 scale=1 1 1
- link left_arm7: geometry collision mesh filename=package://iai_dlr_rollin_justin/mjcf/rollin-justin/meshes/d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 scale=1 1 1; visual mesh filename=package://iai_dlr_rollin_justin/mjcf/rollin-justin/meshes/d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 scale=1 1 1
- link right_1thumb2: geometry collision mesh filename=package://iai_dlr_rollin_justin/mjcf/rollin-justin/meshes/d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 scale=1 1 1; visual mesh filename=package://iai_dlr_rollin_justin/mjcf/rollin-justin/meshes/d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 scale=1 1 1
- link right_1thumb3: geometry collision mesh filename=package://iai_dlr_rollin_justin/mjcf/rollin-justin/meshes/d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 scale=1 1 1; visual mesh filename=package://iai_dlr_rollin_justin/mjcf/rollin-justin/meshes/d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 scale=1 1 1
- link right_1thumb4: geometry collision mesh filename=package://iai_dlr_rollin_justin/mjcf/rollin-justin/meshes/d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 scale=1 1 1; visual mesh filename=package://iai_dlr_rollin_justin/mjcf/rollin-justin/meshes/d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 scale=1 1 1
- link right_1thumb_base: geometry visual mesh filename=package://iai_dlr_rollin_justin/mjcf/rollin-justin/meshes/d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 scale=1 1 1
- link right_2tip2: geometry collision mesh filename=package://iai_dlr_rollin_justin/mjcf/rollin-justin/meshes/d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 scale=1 1 1; visual mesh filename=package://iai_dlr_rollin_justin/mjcf/rollin-justin/meshes/d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 scale=1 1 1
- link right_2tip3: geometry collision mesh filename=package://iai_dlr_rollin_justin/mjcf/rollin-justin/meshes/d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 scale=1 1 1; visual mesh filename=package://iai_dlr_rollin_justin/mjcf/rollin-justin/meshes/d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 scale=1 1 1
- link right_2tip4: geometry collision mesh filename=package://iai_dlr_rollin_justin/mjcf/rollin-justin/meshes/d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 scale=1 1 1; visual mesh filename=package://iai_dlr_rollin_justin/mjcf/rollin-justin/meshes/d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 scale=1 1 1
- link right_2tip_base: geometry visual mesh filename=package://iai_dlr_rollin_justin/mjcf/rollin-justin/meshes/d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 scale=1 1 1
- link right_3middle2: geometry collision mesh filename=package://iai_dlr_rollin_justin/mjcf/rollin-justin/meshes/d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 scale=1 1 1; visual mesh filename=package://iai_dlr_rollin_justin/mjcf/rollin-justin/meshes/d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 scale=1 1 1
- link right_3middle3: geometry collision mesh filename=package://iai_dlr_rollin_justin/mjcf/rollin-justin/meshes/d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 scale=1 1 1; visual mesh filename=package://iai_dlr_rollin_justin/mjcf/rollin-justin/meshes/d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 scale=1 1 1
- link right_3middle4: geometry collision mesh filename=package://iai_dlr_rollin_justin/mjcf/rollin-justin/meshes/d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 scale=1 1 1; visual mesh filename=package://iai_dlr_rollin_justin/mjcf/rollin-justin/meshes/d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 scale=1 1 1
- link right_3middle_base: geometry visual mesh filename=package://iai_dlr_rollin_justin/mjcf/rollin-justin/meshes/d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 scale=1 1 1
- link right_4ring2: geometry collision mesh filename=package://iai_dlr_rollin_justin/mjcf/rollin-justin/meshes/d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 scale=1 1 1; visual mesh filename=package://iai_dlr_rollin_justin/mjcf/rollin-justin/meshes/d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 scale=1 1 1
- link right_4ring3: geometry collision mesh filename=package://iai_dlr_rollin_justin/mjcf/rollin-justin/meshes/d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 scale=1 1 1; visual mesh filename=package://iai_dlr_rollin_justin/mjcf/rollin-justin/meshes/d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 scale=1 1 1
- link right_4ring4: geometry collision mesh filename=package://iai_dlr_rollin_justin/mjcf/rollin-justin/meshes/d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 scale=1 1 1; visual mesh filename=package://iai_dlr_rollin_justin/mjcf/rollin-justin/meshes/d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 scale=1 1 1
- link right_4ring_base: geometry visual mesh filename=package://iai_dlr_rollin_justin/mjcf/rollin-justin/meshes/d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 scale=1 1 1
- link right_arm1: geometry collision mesh filename=package://iai_dlr_rollin_justin/mjcf/rollin-justin/meshes/d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 scale=1 1 1; visual mesh filename=package://iai_dlr_rollin_justin/mjcf/rollin-justin/meshes/d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 scale=1 1 1
- link right_arm2: geometry collision mesh filename=package://iai_dlr_rollin_justin/mjcf/rollin-justin/meshes/d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 scale=1 1 1; visual mesh filename=package://iai_dlr_rollin_justin/mjcf/rollin-justin/meshes/d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 scale=1 1 1
- link right_arm3: geometry collision mesh filename=package://iai_dlr_rollin_justin/mjcf/rollin-justin/meshes/d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 scale=1 1 1; visual mesh filename=package://iai_dlr_rollin_justin/mjcf/rollin-justin/meshes/d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 scale=1 1 1
- link right_arm4: geometry collision mesh filename=package://iai_dlr_rollin_justin/mjcf/rollin-justin/meshes/d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 scale=1 1 1; visual mesh filename=package://iai_dlr_rollin_justin/mjcf/rollin-justin/meshes/d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 scale=1 1 1
- link right_arm5: geometry collision mesh filename=package://iai_dlr_rollin_justin/mjcf/rollin-justin/meshes/d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 scale=1 1 1; visual mesh filename=package://iai_dlr_rollin_justin/mjcf/rollin-justin/meshes/d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 scale=1 1 1
- link right_arm6: geometry collision mesh filename=package://iai_dlr_rollin_justin/mjcf/rollin-justin/meshes/d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 scale=1 1 1; visual mesh filename=package://iai_dlr_rollin_justin/mjcf/rollin-justin/meshes/d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 scale=1 1 1
- link right_arm7: geometry collision mesh filename=package://iai_dlr_rollin_justin/mjcf/rollin-justin/meshes/d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 scale=1 1 1; visual mesh filename=package://iai_dlr_rollin_justin/mjcf/rollin-justin/meshes/d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 scale=1 1 1
- link torso1: geometry collision mesh filename=package://iai_dlr_rollin_justin/mjcf/rollin-justin/meshes/d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 scale=1 1 1; visual mesh filename=package://iai_dlr_rollin_justin/mjcf/rollin-justin/meshes/d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 scale=1 1 1
- link torso2: geometry collision mesh filename=package://iai_dlr_rollin_justin/mjcf/rollin-justin/meshes/d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 scale=1 1 1; visual mesh filename=package://iai_dlr_rollin_justin/mjcf/rollin-justin/meshes/d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 scale=1 1 1
- link torso3: geometry collision mesh filename=package://iai_dlr_rollin_justin/mjcf/rollin-justin/meshes/d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 scale=1 1 1; visual mesh filename=package://iai_dlr_rollin_justin/mjcf/rollin-justin/meshes/d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 scale=1 1 1
- link torso4: geometry collision mesh filename=package://iai_dlr_rollin_justin/mjcf/rollin-justin/meshes/d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 scale=1 1 1; visual mesh filename=package://iai_dlr_rollin_justin/mjcf/rollin-justin/meshes/d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 scale=1 1 1

Commit message: [docker] reverted curl link, and fixed some files for rollin_justin

File: resources/robots/rollin_justin.urdf (robot description, URDF)
Before this commit: robot rollin_justin, 66 links, 65 joints
Links:
- link base_link: geometry collision mesh filename=package://iai_dlr_rollin_justin/mjcf/rollin-justin/meshes/s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 scale=1 1 1; visual mesh filename=package://iai_dlr_rollin_justin/mjcf/rollin-justin/meshes/d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 scale=1 1 1
- link head1: geometry collision mesh filename=package://iai_dlr_rollin_justin/mjcf/rollin-justin/meshes/s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 scale=1 1 1; visual mesh filename=package://iai_dlr_rollin_justin/mjcf/rollin-justin/meshes/d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 scale=1 1 1
- link head2: geometry collision mesh filename=package://iai_dlr_rollin_justin/mjcf/rollin-justin/meshes/s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 scale=1 1 1; visual mesh filename=package://iai_dlr_rollin_justin/mjcf/rollin-justin/meshes/d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 scale=1 1 1
- link left_1thumb2: geometry collision mesh filename=package://iai_dlr_rollin_justin/mjcf/rollin-justin/meshes/s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 scale=1 1 1; visual mesh filename=package://iai_dlr_rollin_justin/mjcf/rollin-justin/meshes/d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 scale=1 1 1
- link left_1thumb3: geometry collision mesh filename=package://iai_dlr_rollin_justin/mjcf/rollin-justin/meshes/s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 scale=1 1 1; visual mesh filename=package://iai_dlr_rollin_justin/mjcf/rollin-justin/meshes/d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 scale=1 1 1
- link left_1thumb4: geometry collision mesh filename=package://iai_dlr_rollin_justin/mjcf/rollin-justin/meshes/s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 scale=1 1 1; visual mesh filename=package://iai_dlr_rollin_justin/mjcf/rollin-justin/meshes/d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 scale=1 1 1
- link left_2tip2: geometry collision mesh filename=package://iai_dlr_rollin_justin/mjcf/rollin-justin/meshes/s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 scale=1 1 1; visual mesh filename=package://iai_dlr_rollin_justin/mjcf/rollin-justin/meshes/d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 scale=1 1 1
- link left_2tip3: geometry collision mesh filename=package://iai_dlr_rollin_justin/mjcf/rollin-justin/meshes/s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 scale=1 1 1; visual mesh filename=package://iai_dlr_rollin_justin/mjcf/rollin-justin/meshes/d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 scale=1 1 1
- link left_2tip4: geometry collision mesh filename=package://iai_dlr_rollin_justin/mjcf/rollin-justin/meshes/s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 scale=1 1 1; visual mesh filename=package://iai_dlr_rollin_justin/mjcf/rollin-justin/meshes/d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 scale=1 1 1
- link left_3middle2: geometry collision mesh filename=package://iai_dlr_rollin_justin/mjcf/rollin-justin/meshes/s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 scale=1 1 1; visual mesh filename=package://iai_dlr_rollin_justin/mjcf/rollin-justin/meshes/d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 scale=1 1 1
- link left_3middle3: geometry collision mesh filename=package://iai_dlr_rollin_justin/mjcf/rollin-justin/meshes/s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 scale=1 1 1; visual mesh filename=package://iai_dlr_rollin_justin/mjcf/rollin-justin/meshes/d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 scale=1 1 1
- link left_3middle4: geometry collision mesh filename=package://iai_dlr_rollin_justin/mjcf/rollin-justin/meshes/s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 scale=1 1 1; visual mesh filename=package://iai_dlr_rollin_justin/mjcf/rollin-justin/meshes/d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 scale=1 1 1
- link left_3middle_base: geometry collision mesh filename=package://iai_dlr_rollin_justin/mjcf/rollin-justin/meshes/s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 scale=1 1 1; visual mesh filename=package://iai_dlr_rollin_justin/mjcf/rollin-justin/meshes/d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 scale=1 1 1
- link left_4ring2: geometry collision mesh filename=package://iai_dlr_rollin_justin/mjcf/rollin-justin/meshes/s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 scale=1 1 1; visual mesh filename=package://iai_dlr_rollin_justin/mjcf/rollin-justin/meshes/d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 scale=1 1 1
- link left_4ring3: geometry collision mesh filename=package://iai_dlr_rollin_justin/mjcf/rollin-justin/meshes/s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 scale=1 1 1; visual mesh filename=package://iai_dlr_rollin_justin/mjcf/rollin-justin/meshes/d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 scale=1 1 1
- link left_4ring4: geometry collision mesh filename=package://iai_dlr_rollin_justin/mjcf/rollin-justin/meshes/s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 scale=1 1 1; visual mesh filename=package://iai_dlr_rollin_justin/mjcf/rollin-justin/meshes/d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 scale=1 1 1
- link left_arm1: geometry collision mesh filename=package://iai_dlr_rollin_justin/mjcf/rollin-justin/meshes/s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 scale=1 1 1; visual mesh filename=package://iai_dlr_rollin_justin/mjcf/rollin-justin/meshes/d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 scale=1 1 1
- link left_arm2: geometry collision mesh filename=package://iai_dlr_rollin_justin/mjcf/rollin-justin/meshes/s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 scale=1 1 1; visual mesh filename=package://iai_dlr_rollin_justin/mjcf/rollin-justin/meshes/d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 scale=1 1 1
- link left_arm3: geometry collision mesh filename=package://iai_dlr_rollin_justin/mjcf/rollin-justin/meshes/s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 scale=1 1 1; visual mesh filename=package://iai_dlr_rollin_justin/mjcf/rollin-justin/meshes/d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 scale=1 1 1
- link left_arm4: geometry collision mesh filename=package://iai_dlr_rollin_justin/mjcf/rollin-justin/meshes/s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 scale=1 1 1; visual mesh filename=package://iai_dlr_rollin_justin/mjcf/rollin-justin/meshes/d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 scale=1 1 1
- link left_arm5: geometry collision mesh filename=package://iai_dlr_rollin_justin/mjcf/rollin-justin/meshes/s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 scale=1 1 1; visual mesh filename=package://iai_dlr_rollin_justin/mjcf/rollin-justin/meshes/d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 scale=1 1 1
- link left_arm6: geometry collision mesh filename=package://iai_dlr_rollin_justin/mjcf/rollin-justin/meshes/s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 scale=1 1 1; visual mesh filename=package://iai_dlr_rollin_justin/mjcf/rollin-justin/meshes/d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 scale=1 1 1
- link left_arm7: geometry collision mesh filename=package://iai_dlr_rollin_justin/mjcf/rollin-justin/meshes/s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 scale=1 1 1; visual mesh filename=package://iai_dlr_rollin_justin/mjcf/rollin-justin/meshes/d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 scale=1 1 1
- link right_1thumb2: geometry collision mesh filename=package://iai_dlr_rollin_justin/mjcf/rollin-justin/meshes/s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 scale=1 1 1; visual mesh filename=package://iai_dlr_rollin_justin/mjcf/rollin-justin/meshes/d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 scale=1 1 1
- link right_1thumb3: geometry collision mesh filename=package://iai_dlr_rollin_justin/mjcf/rollin-justin/meshes/s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 scale=1 1 1; visual mesh filename=package://iai_dlr_rollin_justin/mjcf/rollin-justin/meshes/d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 scale=1 1 1
- link right_1thumb4: geometry collision mesh filename=package://iai_dlr_rollin_justin/mjcf/rollin-justin/meshes/s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 scale=1 1 1; visual mesh filename=package://iai_dlr_rollin_justin/mjcf/rollin-justin/meshes/d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 scale=1 1 1
- link right_2tip2: geometry collision mesh filename=package://iai_dlr_rollin_justin/mjcf/rollin-justin/meshes/s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 scale=1 1 1; visual mesh filename=package://iai_dlr_rollin_justin/mjcf/rollin-justin/meshes/d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 scale=1 1 1
- link right_2tip3: geometry collision mesh filename=package://iai_dlr_rollin_justin/mjcf/rollin-justin/meshes/s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 scale=1 1 1; visual mesh filename=package://iai_dlr_rollin_justin/mjcf/rollin-justin/meshes/d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 scale=1 1 1
- link right_2tip4: geometry collision mesh filename=package://iai_dlr_rollin_justin/mjcf/rollin-justin/meshes/s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 scale=1 1 1; visual mesh filename=package://iai_dlr_rollin_justin/mjcf/rollin-justin/meshes/d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 scale=1 1 1
- link right_3middle2: geometry collision mesh filename=package://iai_dlr_rollin_justin/mjcf/rollin-justin/meshes/s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 scale=1 1 1; visual mesh filename=package://iai_dlr_rollin_justin/mjcf/rollin-justin/meshes/d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 scale=1 1 1
- link right_3middle3: geometry collision mesh filename=package://iai_dlr_rollin_justin/mjcf/rollin-justin/meshes/s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 scale=1 1 1; visual mesh filename=package://iai_dlr_rollin_justin/mjcf/rollin-justin/meshes/d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 scale=1 1 1
- link right_3middle4: geometry collision mesh filename=package://iai_dlr_rollin_justin/mjcf/rollin-justin/meshes/s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 scale=1 1 1; visual mesh filename=package://iai_dlr_rollin_justin/mjcf/rollin-justin/meshes/d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 scale=1 1 1
- link right_4ring2: geometry collision mesh filename=package://iai_dlr_rollin_justin/mjcf/rollin-justin/meshes/s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 scale=1 1 1; visual mesh filename=package://iai_dlr_rollin_justin/mjcf/rollin-justin/meshes/d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 scale=1 1 1
- link right_4ring3: geometry collision mesh filename=package://iai_dlr_rollin_justin/mjcf/rollin-justin/meshes/s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 scale=1 1 1; visual mesh filename=package://iai_dlr_rollin_justin/mjcf/rollin-justin/meshes/d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 scale=1 1 1
- link right_4ring4: geometry collision mesh filename=package://iai_dlr_rollin_justin/mjcf/rollin-justin/meshes/s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 scale=1 1 1; visual mesh filename=package://iai_dlr_rollin_justin/mjcf/rollin-justin/meshes/d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 scale=1 1 1
- link right_arm1: geometry collision mesh filename=package://iai_dlr_rollin_justin/mjcf/rollin-justin/meshes/s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 scale=1 1 1; visual mesh filename=package://iai_dlr_rollin_justin/mjcf/rollin-justin/meshes/d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 scale=1 1 1
- link right_arm2: geometry collision mesh filename=package://iai_dlr_rollin_justin/mjcf/rollin-justin/meshes/s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 scale=1 1 1; visual mesh filename=package://iai_dlr_rollin_justin/mjcf/rollin-justin/meshes/d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 scale=1 1 1
- link right_arm3: geometry collision mesh filename=package://iai_dlr_rollin_justin/mjcf/rollin-justin/meshes/s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 scale=1 1 1; visual mesh filename=package://iai_dlr_rollin_justin/mjcf/rollin-justin/meshes/d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 scale=1 1 1
- link right_arm4: geometry collision mesh filename=package://iai_dlr_rollin_justin/mjcf/rollin-justin/meshes/s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 scale=1 1 1; visual mesh filename=package://iai_dlr_rollin_justin/mjcf/rollin-justin/meshes/d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 scale=1 1 1
- link right_arm5: geometry collision mesh filename=package://iai_dlr_rollin_justin/mjcf/rollin-justin/meshes/s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 scale=1 1 1; visual mesh filename=package://iai_dlr_rollin_justin/mjcf/rollin-justin/meshes/d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 scale=1 1 1
- link right_arm6: geometry collision mesh filename=package://iai_dlr_rollin_justin/mjcf/rollin-justin/meshes/s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 scale=1 1 1; visual mesh filename=package://iai_dlr_rollin_justin/mjcf/rollin-justin/meshes/d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 scale=1 1 1
- link right_arm7: geometry collision mesh filename=package://iai_dlr_rollin_justin/mjcf/rollin-justin/meshes/s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 scale=1 1 1; visual mesh filename=package://iai_dlr_rollin_justin/mjcf/rollin-justin/meshes/d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 scale=1 1 1
- link torso1: geometry collision mesh filename=package://iai_dlr_rollin_justin/mjcf/rollin-justin/meshes/s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 scale=1 1 1; visual mesh filename=package://iai_dlr_rollin_justin/mjcf/rollin-justin/meshes/d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 scale=1 1 1
- link torso2: geometry collision mesh filename=package://iai_dlr_rollin_justin/mjcf/rollin-justin/meshes/s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 scale=1 1 1; visual mesh filename=package://iai_dlr_rollin_justin/mjcf/rollin-justin/meshes/d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 scale=1 1 1
- link torso3: geometry collision mesh filename=package://iai_dlr_rollin_justin/mjcf/rollin-justin/meshes/s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 scale=1 1 1; visual mesh filename=package://iai_dlr_rollin_justin/mjcf/rollin-justin/meshes/d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 scale=1 1 1
- link torso4: geometry collision mesh filename=package://iai_dlr_rollin_justin/mjcf/rollin-justin/meshes/s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 scale=1 1 1; visual mesh filename=package://iai_dlr_rollin_justin/mjcf/rollin-justin/meshes/d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 scale=1 1 1
