Commit message: [tiago] integrated tiago into the new binder structure

File: resources/robots/tiago_dual.urdf (robot description, URDF)
Before this commit: robot tiago_dual, 69 links, 68 joints
Joints:
- joint gripper_left_tool_joint: origin xyz=0.01 0 0 rpy=1.5707963267948966 1.5707963267948966 -1.5707963267948966 -> xyz=0.18 0 0 rpy=1.5707963267948966 1.5707963267948966 -1.5707963267948966
- joint gripper_right_tool_joint: origin xyz=0.01 0 0 rpy=1.5707963267948966 1.5707963267948966 -1.5707963267948966 -> xyz=0.18 0 0 rpy=1.5707963267948966 1.5707963267948966 -1.5707963267948966
