Commit message: [feature] first test icub on pybullet

File: resources/robots/icub.urdf (robot description, URDF)
Before this commit: robot iCub, 102 links, 101 joints
Links:
- link chest: geometry collision mesh filename=package://icub_model/meshes/simmechanics/sim_sea_2-5_chest_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 scale=0.001 0.001 0.001; visual mesh filename=package://icub_model/meshes/simmechanics/sim_sea_2-5_chest_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 scale=0.001 0.001 0.001
- link head: geometry collision mesh filename=package://icub_model/meshes/simmechanics/sim_sea_2-5_head_p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 scale=0.001 0.001 0.001; visual mesh filename=package://icub_model/meshes/simmechanics/sim_sea_2-5_head_p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 scale=0.001 0.001 0.001
- link l_ankle_1: geometry collision mesh filename=package://icub_model/meshes/simmechanics/sim_sea_2-5_l_ankl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 scale=0.001 0.001 0.001; visual mesh filename=package://icub_model/meshes/simmechanics/sim_sea_2-5_l_ankl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 scale=0.001 0.001 0.001
- link l_ankle_2: geometry collision mesh filename=package://icub_model/meshes/simmechanics/sim_sea_2-5_l_foot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 scale=0.001 0.001 0.001; visual mesh filename=package://icub_model/meshes/simmechanics/sim_sea_2-5_l_foot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 scale=0.001 0.001 0.001
- link l_elbow_1: geometry collision mesh filename=package://icub_model/meshes/simmechanics/sim_sea_2-5_l_elbo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 scale=0.001 0.001 0.001; visual mesh filename=package://icub_model/meshes/simmechanics/sim_sea_2-5_l_elbo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 scale=0.001 0.001 0.001
- link l_foot: geometry collision box size=0.16 0.072 0.001; visual mesh filename=package://icub_model/meshes/simmechanics/sim_sea_2-5_l_sole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 scale=0.001 0.001 0.001
- link l_forearm: geometry collision mesh filename=package://icub_model/meshes/simmechanics/sim_sea_2-5_l_fore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 scale=0.001 0.001 0.001; visual mesh filename=package://icub_model/meshes/simmechanics/sim_sea_2-5_l_fore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 scale=0.001 0.001 0.001
- link l_hand: geometry collision mesh filename=package://icub_model/meshes/col_LeftHandPalm.dae scale=1.0 1.0 1.0; visual mesh filename=package://icub_model/meshes/full_LeftHandPalm.dae scale=1.0 1.0 1.0
- link l_hand_index_0: geometry collision mesh filename=package://icub_model/meshes/col_LeftIndex0.dae scale=1.0 1.0 1.0; visual mesh filename=package://icub_model/meshes/full_LeftIndex0.dae scale=1.0 1.0 1.0
- link l_hand_index_1: geometry collision mesh filename=package://icub_model/meshes/col_LeftIndex1.dae scale=1.0 1.0 1.0; visual mesh filename=package://icub_model/meshes/full_LeftIndex1.dae scale=1.0 1.0 1.0
- link l_hand_index_2: geometry collision mesh filename=package://icub_model/meshes/col_LeftIndex2.dae scale=1.0 1.0 1.0; visual mesh filename=package://icub_model/meshes/full_LeftIndex2.dae scale=1.0 1.0 1.0
- link l_hand_index_3: geometry collision mesh filename=package://icub_model/meshes/col_LeftIndex3.dae scale=1.0 1.0 1.0; visual mesh filename=package://icub_model/meshes/full_LeftIndex3.dae scale=1.0 1.0 1.0
- link l_hand_little_0: geometry collision mesh filename=package://icub_model/meshes/col_LeftLittle0.dae scale=1.0 1.0 1.0; visual mesh filename=package://icub_model/meshes/full_LeftLittle0.dae scale=1.0 1.0 1.0
- link l_hand_little_1: geometry collision mesh filename=package://icub_model/meshes/col_LeftLittle1.dae scale=1.0 1.0 1.0; visual mesh filename=package://icub_model/meshes/full_LeftLittle1.dae scale=1.0 1.0 1.0
- link l_hand_little_2: geometry collision mesh filename=package://icub_model/meshes/col_LeftLittle2.dae scale=1.0 1.0 1.0; visual mesh filename=package://icub_model/meshes/full_LeftLittle2.dae scale=1.0 1.0 1.0
- link l_hand_little_3: geometry collision mesh filename=package://icub_model/meshes/col_LeftLittle3.dae scale=1.0 1.0 1.0; visual mesh filename=package://icub_model/meshes/full_LeftLittle3.dae scale=1.0 1.0 1.0
- link l_hand_middle_0: geometry collision mesh filename=package://icub_model/meshes/col_LeftMiddle0.dae scale=1.0 1.0 1.0; visual mesh filename=package://icub_model/meshes/full_LeftMiddle0.dae scale=1.0 1.0 1.0
- link l_hand_middle_1: geometry collision mesh filename=package://icub_model/meshes/col_LeftMiddle1.dae scale=1.0 1.0 1.0; visual mesh filename=package://icub_model/meshes/full_LeftMiddle1.dae scale=1.0 1.0 1.0
- link l_hand_middle_2: geometry collision mesh filename=package://icub_model/meshes/col_LeftMiddle2.dae scale=1.0 1.0 1.0; visual mesh filename=package://icub_model/meshes/full_LeftMiddle2.dae scale=1.0 1.0 1.0
- link l_hand_middle_3: geometry collision mesh filename=package://icub_model/meshes/col_LeftMiddle3.dae scale=1.0 1.0 1.0; visual mesh filename=package://icub_model/meshes/full_LeftMiddle3.dae scale=1.0 1.0 1.0
- link l_hand_ring_0: geometry collision mesh filename=package://icub_model/meshes/col_LeftRing0.dae scale=1.0 1.0 1.0; visual mesh filename=package://icub_model/meshes/full_LeftRing0.dae scale=1.0 1.0 1.0
- link l_hand_ring_1: geometry collision mesh filename=package://icub_model/meshes/col_LeftRing1.dae scale=1.0 1.0 1.0; visual mesh filename=package://icub_model/meshes/full_LeftRing1.dae scale=1.0 1.0 1.0
- link l_hand_ring_2: geometry collision mesh filename=package://icub_model/meshes/col_LeftRing2.dae scale=1.0 1.0 1.0; visual mesh filename=package://icub_model/meshes/full_LeftRing2.dae scale=1.0 1.0 1.0
- link l_hand_ring_3: geometry collision mesh filename=package://icub_model/meshes/col_LeftRing3.dae scale=1.0 1.0 1.0; visual mesh filename=package://icub_model/meshes/full_LeftRing3.dae scale=1.0 1.0 1.0
- link l_hand_thumb_0: geometry collision mesh filename=package://icub_model/meshes/col_LeftThumb0.dae scale=1.0 1.0 1.0; visual mesh filename=package://icub_model/meshes/full_LeftThumb0.dae scale=1.0 1.0 1.0
- link l_hand_thumb_1: geometry collision mesh filename=package://icub_model/meshes/col_LeftThumb1.dae scale=1.0 1.0 1.0; visual mesh filename=package://icub_model/meshes/full_LeftThumb1.dae scale=1.0 1.0 1.0
- link l_hand_thumb_2: geometry collision mesh filename=package://icub_model/meshes/col_LeftThumb2.dae scale=1.0 1.0 1.0; visual mesh filename=package://icub_model/meshes/full_LeftThumb2.dae scale=1.0 1.0 1.0
- link l_hand_thumb_3: geometry collision mesh filename=package://icub_model/meshes/col_LeftThumb3.dae scale=1.0 1.0 1.0; visual mesh filename=package://icub_model/meshes/full_LeftThumb3.dae scale=1.0 1.0 1.0
- link l_hip_1: geometry collision mesh filename=package://icub_model/meshes/simmechanics/sim_sea_2-5_l_hip_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 scale=0.001 0.001 0.001; visual mesh filename=package://icub_model/meshes/simmechanics/sim_sea_2-5_l_hip_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 scale=0.001 0.001 0.001
- link l_hip_2: geometry collision mesh filename=package://icub_model/meshes/simmechanics/sim_sea_2-5_l_hip_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 scale=0.001 0.001 0.001; visual mesh filename=package://icub_model/meshes/simmechanics/sim_sea_2-5_l_hip_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 scale=0.001 0.001 0.001
- link l_hip_3: geometry collision mesh filename=package://icub_model/meshes/simmechanics/sim_sea_2-5_l_uppe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 scale=0.001 0.001 0.001; visual mesh filename=package://icub_model/meshes/simmechanics/sim_sea_2-5_l_uppe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 scale=0.001 0.001 0.001
- link l_lower_leg: geometry collision mesh filename=package://icub_model/meshes/simmechanics/sim_sea_2-5_l_shan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 scale=0.001 0.001 0.001; visual mesh filename=package://icub_model/meshes/simmechanics/sim_sea_2-5_l_shan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 scale=0.001 0.001 0.001
- link l_shoulder_1: geometry collision mesh filename=package://icub_model/meshes/simmechanics/sim_sea_2-5_l_shou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 scale=0.001 0.001 0.001; visual mesh filename=package://icub_model/meshes/simmechanics/sim_sea_2-5_l_shou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 scale=0.001 0.001 0.001
- link l_shoulder_2: geometry collision mesh filename=package://icub_model/meshes/simmechanics/sim_sea_2-5_l_shou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 scale=0.001 0.001 0.001; visual mesh filename=package://icub_model/meshes/simmechanics/sim_sea_2-5_l_shou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 scale=0.001 0.001 0.001
- link l_shoulder_3: geometry collision mesh filename=package://icub_model/meshes/simmechanics/sim_sea_2-5_l_uppe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 scale=0.001 0.001 0.001; visual mesh filename=package://icub_model/meshes/simmechanics/sim_sea_2-5_l_uppe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 scale=0.001 0.001 0.001
- link l_upper_arm: geometry collision mesh filename=package://icub_model/meshes/simmechanics/sim_sea_2-5_l_elbo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 scale=0.001 0.001 0.001; visual mesh filename=package://icub_model/meshes/simmechanics/sim_sea_2-5_l_elbo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 scale=0.001 0.001 0.001
- link l_upper_leg: geometry collision mesh filename=package://icub_model/meshes/simmechanics/sim_sea_2-5_l_thig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 scale=0.001 0.001 0.001; visual mesh filename=package://icub_model/meshes/simmechanics/sim_sea_2-5_l_thig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 scale=0.001 0.001 0.001
- link l_wrist_1: geometry collision mesh filename=package://icub_model/meshes/simmechanics/sim_sea_2-5_l_wris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 scale=0.001 0.001 0.001; visual mesh filename=package://icub_model/meshes/simmechanics/sim_sea_2-5_l_wris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 scale=0.001 0.001 0.001
- link neck_1: geometry collision mesh filename=package://icub_model/meshes/simmechanics/sim_sea_2-5_neck_1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 scale=0.001 0.001 0.001; visual mesh filename=package://icub_model/meshes/simmechanics/sim_sea_2-5_neck_1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 scale=0.001 0.001 0.001
- link neck_2: geometry collision mesh filename=package://icub_model/meshes/simmechanics/sim_sea_2-5_neck_2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 scale=0.001 0.001 0.001; visual mesh filename=package://icub_model/meshes/simmechanics/sim_sea_2-5_neck_2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 scale=0.001 0.001 0.001
- link r_ankle_1: geometry collision mesh filename=package://icub_model/meshes/simmechanics/sim_sea_2-5_r_ankl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 scale=0.001 0.001 0.001; visual mesh filename=package://icub_model/meshes/simmechanics/sim_sea_2-5_r_ankl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 scale=0.001 0.001 0.001
- link r_ankle_2: geometry collision mesh filename=package://icub_model/meshes/simmechanics/sim_sea_2-5_r_foot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 scale=0.001 0.001 0.001; visual mesh filename=package://icub_model/meshes/simmechanics/sim_sea_2-5_r_foot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 scale=0.001 0.001 0.001
- link r_elbow_1: geometry collision mesh filename=package://icub_model/meshes/simmechanics/sim_sea_2-5_r_elbo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 scale=0.001 0.001 0.001; visual mesh filename=package://icub_model/meshes/simmechanics/sim_sea_2-5_r_elbo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 scale=0.001 0.001 0.001
- link r_foot: geometry collision box size=0.16 0.072 0.001; visual mesh filename=package://icub_model/meshes/simmechanics/sim_sea_2-5_r_sole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 scale=0.001 0.001 0.001
- link r_forearm: geometry collision mesh filename=package://icub_model/meshes/simmechanics/sim_sea_2-5_r_fore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 scale=0.001 0.001 0.001; visual mesh filename=package://icub_model/meshes/simmechanics/sim_sea_2-5_r_fore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 scale=0.001 0.001 0.001
- link r_hand: geometry collision mesh filename=package://icub_model/meshes/col_RightHandPalm.dae scale=1.0 1.0 1.0; visual mesh filename=package://icub_model/meshes/full_RightHandPalm.dae scale=1.0 1.0 1.0
- link r_hand_index_0: geometry collision mesh filename=package://icub_model/meshes/col_RightIndex0.dae scale=1.0 1.0 1.0; visual mesh filename=package://icub_model/meshes/full_RightIndex0.dae scale=1.0 1.0 1.0
- link r_hand_index_1: geometry collision mesh filename=package://icub_model/meshes/col_RightIndex1.dae scale=1.0 1.0 1.0; visual mesh filename=package://icub_model/meshes/full_RightIndex1.dae scale=1.0 1.0 1.0
- link r_hand_index_2: geometry collision mesh filename=package://icub_model/meshes/col_RightIndex2.dae scale=1.0 1.0 1.0; visual mesh filename=package://icub_model/meshes/full_RightIndex2.dae scale=1.0 1.0 1.0
- link r_hand_index_3: geometry collision mesh filename=package://icub_model/meshes/col_RightIndex3.dae scale=1.0 1.0 1.0; visual mesh filename=package://icub_model/meshes/full_RightIndex3.dae scale=1.0 1.0 1.0
- link r_hand_little_0: geometry collision mesh filename=package://icub_model/meshes/col_RightLittle0.dae scale=1.0 1.0 1.0; visual mesh filename=package://icub_model/meshes/full_RightLittle0.dae scale=1.0 1.0 1.0
- link r_hand_little_1: geometry collision mesh filename=package://icub_model/meshes/col_RightLittle1.dae scale=1.0 1.0 1.0; visual mesh filename=package://icub_model/meshes/full_RightLittle1.dae scale=1.0 1.0 1.0
- link r_hand_little_2: geometry collision mesh filename=package://icub_model/meshes/col_RightLittle2.dae scale=1.0 1.0 1.0; visual mesh filename=package://icub_model/meshes/full_RightLittle2.dae scale=1.0 1.0 1.0
- link r_hand_little_3: geometry collision mesh filename=package://icub_model/meshes/col_RightLittle3.dae scale=1.0 1.0 1.0; visual mesh filename=package://icub_model/meshes/full_RightLittle3.dae scale=1.0 1.0 1.0
- link r_hand_middle_0: geometry collision mesh filename=package://icub_model/meshes/col_RightMiddle0.dae scale=1.0 1.0 1.0; visual mesh filename=package://icub_model/meshes/full_RightMiddle0.dae scale=1.0 1.0 1.0
- link r_hand_middle_1: geometry collision mesh filename=package://icub_model/meshes/col_RightMiddle1.dae scale=1.0 1.0 1.0; visual mesh filename=package://icub_model/meshes/full_RightMiddle1.dae scale=1.0 1.0 1.0
- link r_hand_middle_2: geometry collision mesh filename=package://icub_model/meshes/col_RightMiddle2.dae scale=1.0 1.0 1.0; visual mesh filename=package://icub_model/meshes/full_RightMiddle2.dae scale=1.0 1.0 1.0
- link r_hand_middle_3: geometry collision mesh filename=package://icub_model/meshes/col_RightMiddle3.dae scale=1.0 1.0 1.0; visual mesh filename=package://icub_model/meshes/full_RightMiddle3.dae scale=1.0 1.0 1.0
- link r_hand_ring_0: geometry collision mesh filename=package://icub_model/meshes/col_RightRing0.dae scale=1.0 1.0 1.0; visual mesh filename=package://icub_model/meshes/full_RightRing0.dae scale=1.0 1.0 1.0
- link r_hand_ring_1: geometry collision mesh filename=package://icub_model/meshes/col_RightRing1.dae scale=1.0 1.0 1.0; visual mesh filename=package://icub_model/meshes/full_RightRing1.dae scale=1.0 1.0 1.0
- link r_hand_ring_2: geometry collision mesh filename=package://icub_model/meshes/col_RightRing2.dae scale=1.0 1.0 1.0; visual mesh filename=package://icub_model/meshes/full_RightRing2.dae scale=1.0 1.0 1.0
- link r_hand_ring_3: geometry collision mesh filename=package://icub_model/meshes/col_RightRing3.dae scale=1.0 1.0 1.0; visual mesh filename=package://icub_model/meshes/full_RightRing3.dae scale=1.0 1.0 1.0
- link r_hand_thumb_0: geometry collision mesh filename=package://icub_model/meshes/col_RightThumb0.dae scale=1.0 1.0 1.0; visual mesh filename=package://icub_model/meshes/full_RightThumb0.dae scale=1.0 1.0 1.0
- link r_hand_thumb_1: geometry collision mesh filename=package://icub_model/meshes/col_RightThumb1.dae scale=1.0 1.0 1.0; visual mesh filename=package://icub_model/meshes/full_RightThumb1.dae scale=1.0 1.0 1.0
- link r_hand_thumb_2: geometry collision mesh filename=package://icub_model/meshes/col_RightThumb2.dae scale=1.0 1.0 1.0; visual mesh filename=package://icub_model/meshes/full_RightThumb2.dae scale=1.0 1.0 1.0
- link r_hand_thumb_3: geometry collision mesh filename=package://icub_model/meshes/col_RightThumb3.dae scale=1.0 1.0 1.0; visual mesh filename=package://icub_model/meshes/full_RightThumb3.dae scale=1.0 1.0 1.0
- link r_hip_1: geometry collision mesh filename=package://icub_model/meshes/simmechanics/sim_sea_2-5_r_hip_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 scale=0.001 0.001 0.001; visual mesh filename=package://icub_model/meshes/simmechanics/sim_sea_2-5_r_hip_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 scale=0.001 0.001 0.001
- link r_hip_2: geometry collision mesh filename=package://icub_model/meshes/simmechanics/sim_sea_2-5_r_hip_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 scale=0.001 0.001 0.001; visual mesh filename=package://icub_model/meshes/simmechanics/sim_sea_2-5_r_hip_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 scale=0.001 0.001 0.001
- link r_hip_3: geometry collision mesh filename=package://icub_model/meshes/simmechanics/sim_sea_2-5_r_uppe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 scale=0.001 0.001 0.001; visual mesh filename=package://icub_model/meshes/simmechanics/sim_sea_2-5_r_uppe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 scale=0.001 0.001 0.001
- link r_lower_leg: geometry collision mesh filename=package://icub_model/meshes/simmechanics/sim_sea_2-5_r_shan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 scale=0.001 0.001 0.001; visual mesh filename=package://icub_model/meshes/simmechanics/sim_sea_2-5_r_shan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 scale=0.001 0.001 0.001
- link r_shoulder_1: geometry collision mesh filename=package://icub_model/meshes/simmechanics/sim_sea_2-5_r_shou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 scale=0.001 0.001 0.001; visual mesh filename=package://icub_model/meshes/simmechanics/sim_sea_2-5_r_shou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 scale=0.001 0.001 0.001
- link r_shoulder_2: geometry collision mesh filename=package://icub_model/meshes/simmechanics/sim_sea_2-5_r_shou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 scale=0.001 0.001 0.001; visual mesh filename=package://icub_model/meshes/simmechanics/sim_sea_2-5_r_shou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 scale=0.001 0.001 0.001
- link r_shoulder_3: geometry collision mesh filename=package://icub_model/meshes/simmechanics/sim_sea_2-5_r_uppe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 scale=0.001 0.001 0.001; visual mesh filename=package://icub_model/meshes/simmechanics/sim_sea_2-5_r_uppe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 scale=0.001 0.001 0.001
- link r_upper_arm: geometry collision mesh filename=package://icub_model/meshes/simmechanics/sim_sea_2-5_r_elbo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 scale=0.001 0.001 0.001; visual mesh filename=package://icub_model/meshes/simmechanics/sim_sea_2-5_r_elbo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 scale=0.001 0.001 0.001
- link r_upper_leg: geometry collision mesh filename=package://icub_model/meshes/simmechanics/sim_sea_2-5_r_thig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 scale=0.001 0.001 0.001; visual mesh filename=package://icub_model/meshes/simmechanics/sim_sea_2-5_r_thig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 scale=0.001 0.001 0.001
- link r_wrist_1: geometry collision mesh filename=package://icub_model/meshes/simmechanics/sim_sea_2-5_r_wris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 scale=0.001 0.001 0.001; visual mesh filename=package://icub_model/meshes/simmechanics/sim_sea_2-5_r_wris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 scale=0.001 0.001 0.001
- link root_link: geometry collision mesh filename=package://icub_model/meshes/simmechanics/sim_sea_2-5_root_l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 scale=0.001 0.001 0.001; visual mesh filename=package://icub_model/meshes/simmechanics/sim_sea_2-5_root_l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 scale=0.001 0.001 0.001
- link torso_1: geometry collision mesh filename=package://icub_model/meshes/simmechanics/sim_sea_2-5_lap_be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 scale=0.001 0.001 0.001; visual mesh filename=package://icub_model/meshes/simmechanics/sim_sea_2-5_lap_be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 scale=0.001 0.001 0.001
- link torso_2: geometry collision mesh filename=package://icub_model/meshes/simmechanics/sim_sea_2-5_lap_be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 scale=0.001 0.001 0.001; visual mesh filename=package://icub_model/meshes/simmechanics/sim_sea_2-5_lap_be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 scale=0.001 0.001 0.001
