Commit message: [mediator-robot] Cleaned up processmodules, added way to specify yaw/pitch/roll joint in neck, and generalized defaultmovehead and donbotmovehead process modules.

File: resources/robots/iai_donbot.urdf (robot description, URDF)
Before this commit: robot iai_donbot, 44 links, 43 joints
Links:
- removed link odom
- removed link odom_x_frame
- removed link odom_y_frame
- added link wheel_back_left, mass 2.0; collision cylinder length=0.08 radius=0.105; visual mesh filename=package://iai_boxy_base_2/meshes/wheel_back_left.stl
- added link wheel_back_right, mass 2.0; collision cylinder length=0.08 radius=0.105; visual mesh filename=package://iai_boxy_base_2/meshes/wheel_back_right.stl
- added link wheel_front_left, mass 2.0; collision cylinder length=0.08 radius=0.105; visual mesh filename=package://iai_boxy_base_2/meshes/wheel_front_left.stl
- added link wheel_front_right, mass 2.0; collision cylinder length=0.08 radius=0.105; visual mesh filename=package://iai_boxy_base_2/meshes/wheel_front_right.stl
- link adapter_fwa050_wsg50_frame_in: geometry collision mesh filename=package://iai_adapters_description/meshes/adapter_fwa050_ws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 scale=0.001 0.001 0.001; visual mesh filename=package://iai_adapters_description/meshes/adapter_fwa050_ws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 scale=0.001 0.001 0.001
- link adapter_iso50_kms40_frame_in: geometry collision mesh filename=package://iai_kms_40_description/meshes/adapter_plate_iso50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 scale=0.001 0.001 0.001; visual mesh filename=package://iai_kms_40_description/meshes/adapter_plate_iso50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 scale=0.001 0.001 0.001
- link adapter_kms40_fwk050_frame_in: geometry collision mesh filename=package://iai_adapters_description/meshes/adapter_kms40_fwk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 scale=0.001 0.001 0.001; visual mesh filename=package://iai_adapters_description/meshes/adapter_kms40_fwk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 scale=0.001 0.001 0.001
- link base_link: geometry collision mesh filename=package://iai_boxy_base_2/meshes/base_without_wheels_lowres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; visual mesh filename=package://iai_boxy_base_2/meshes/base_without_wheels.stl
- link fwk_fwa_050_frame_in: geometry collision mesh filename=package://iai_adapters_description/meshes/fwk_fwa_050_simpl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 scale=0.001 0.001 0.001; visual mesh filename=package://iai_adapters_description/meshes/fwk_fwa_050_simpl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 scale=0.001 0.001 0.001
- link kms40_frame_in: geometry collision mesh filename=package://iai_kms_40_description/meshes/kms40_simple.stl scale=0.001 0.001 0.001; visual mesh filename=package://iai_kms_40_description/meshes/kms40_simple.stl scale=0.001 0.001 0.001
Joints:
- removed joint odom_x_joint
- removed joint odom_y_joint
- removed joint odom_z_joint
- added joint wheel_back_left_joint: type revolute, parent base_link, child wheel_back_left, origin xyz=-0.648 0.09 -0.06 rpy=0.0 0.0 0.0, axis 0 1 0, limit lower=-1000.0 upper=1000.0 effort=200.0 velocity=1.0
- added joint wheel_back_right_joint: type revolute, parent base_link, child wheel_back_right, origin xyz=-0.648 -0.545 -0.06 rpy=0.0 0.0 0.0, axis 0 1 0, limit lower=-1000.0 upper=1000.0 effort=200.0 velocity=1.0
- added joint wheel_front_left_joint: type revolute, parent base_link, child wheel_front_left, origin xyz=0.13 0.09 -0.06 rpy=0.0 0.0 0.0, axis 0 1 0, limit lower=-1000.0 upper=1000.0 effort=200.0 velocity=1.0
- added joint wheel_front_right_joint: type revolute, parent base_link, child wheel_front_right, origin xyz=0.13 -0.545 -0.06 rpy=0.0 0.0 0.0, axis 0 1 0, limit lower=-1000.0 upper=1000.0 effort=200.0 velocity=1.0
- joint adapter_iso50_kms40_joint: origin xyz=0 0 0 rpy=0 0 3.14159265359 -> xyz=0 0 0 rpy=0 0 3.141592653589793
- joint gripper_to_camera_holder_joint: origin xyz=0 0 0 rpy=0 0 3.14159265359 -> xyz=0 0 0 rpy=0 0 3.141592653589793
- joint gripper_to_camera_joint: origin xyz=0.002956 -0.066498 0.060947 rpy=0.204429 6.281375 3.127197 -> xyz=0.0013289 -0.06619 0.031583 rpy=0.231224 -0.0034913 -3.134637307
- joint kms_mounting_plate_joint: origin xyz=0 0 0 rpy=0 1.57079632679 0 -> xyz=0 0 0 rpy=0 1.5707963267948966 0
- joint ur5_base_link-base_fixed_joint: origin xyz=0 0 0 rpy=0 0 -3.14159265359 -> xyz=0 0 0 rpy=0 0 -3.141592653589793
- joint ur5_ee_fixed_joint: origin xyz=0.0 0.0 0.0 rpy=0.0 -1.57079632679 1.57079632679 -> xyz=0.0 0.0 0.0 rpy=0.0 -1.5707963267948966 1.5707963267948966
- joint ur5_elbow_joint: limit lower=-3.14159265359 upper=3.14159265359 effort=150.0 velocity=3.15 -> lower=-3.141592653589793 upper=3.141592653589793 effort=150.0 velocity=3.15; origin xyz=-0.424875903105 0 0 rpy=3.14141093572 3.14049876452 3.14154086296 -> xyz=-0.425 0 0 rpy=0 0 0
- joint ur5_shoulder_lift_joint: limit lower=-6.28318530718 upper=6.28318530718 effort=150.0 velocity=3.15 -> lower=-6.283185307179586 upper=6.283185307179586 effort=150.0 velocity=3.15; origin xyz=0.000371267234471 0 0 rpy=1.56968458582 0 -5.52038697331e-05 -> xyz=0 0 0 rpy=1.570796327 0 0
- joint ur5_shoulder_pan_joint: limit lower=-6.28318530718 upper=6.28318530718 effort=150.0 velocity=3.15 -> lower=-6.283185307179586 upper=6.283185307179586 effort=150.0 velocity=3.15; origin xyz=0 0 0.0889259622293 rpy=0 0 3.14151729445 -> xyz=0 0 0.089159 rpy=0 0 3.141592653589793
- joint ur5_wrist_1_joint: limit lower=-6.28318530718 upper=6.28318530718 effort=28.0 velocity=3.2 -> lower=-6.283185307179586 upper=6.283185307179586 effort=28.0 velocity=3.2; origin xyz=-0.391622303288 -0.000954289022315 0.111506051949 rpy=0.00855797249115 0.00564631791456 -4.73161394588e-06 -> xyz=-0.39225 0 0.10915 rpy=0 0 0
- joint ur5_wrist_2_joint: limit lower=-6.28318530718 upper=6.28318530718 effort=28.0 velocity=3.2 -> lower=-6.283185307179586 upper=6.283185307179586 effort=28.0 velocity=3.2; origin xyz=-0.000124234587642 -0.0947812268782 6.23931257156e-06 rpy=1.57073049823 0 -2.51013751161e-05 -> xyz=0 -0.09465 -1.941303950897609e-11 rpy=1.570796327 0 0
- joint ur5_wrist_3_joint: limit lower=-6.28318530718 upper=6.28318530718 effort=28.0 velocity=3.2 -> lower=-6.283185307179586 upper=6.283185307179586 effort=28.0 velocity=3.2; origin xyz=7.00453011326e-05 0.0825471455322 -2.54792324043e-05 rpy=1.57048766401 3.14159265359 -3.14158821505 -> xyz=0 0.0823 -1.688001216681175e-11 rpy=1.570796326589793 3.141592653589793 3.141592653589793
- joint wristcam_to_realsense_joint: origin xyz=-0.017993 -0.107556 0.017699 rpy=6.270618 4.930698 1.578454 -> xyz=-0.018594 -0.105693 0.017161 rpy=-0.0120443 -1.3424873 1.579879
