Commit message: new tracy.urdf that is compatible with the one used by giskard + small fixes to robot_state_updater.py

File: resources/robots/tracy.urdf (robot description, URDF)
Before this commit: robot tracy, 51 links, 50 joints
Links:
- removed link world
- added link left_world
- added link map
- added link right_world
Joints:
- added joint left_world_joint: type fixed, parent left_arm_mount, child left_world, origin xyz=0.0 0.0 0.0 rpy=0.0 0.0 3.141592653589793
- added joint right_world_joint: type fixed, parent right_arm_mount, child right_world, origin xyz=0.0 0.0 0.0 rpy=0.0 0.0 0.0
- joint l_gripper_tool_frame_joint: origin xyz=0.0 0.0 0.144 rpy=0.0 -1.57079632679 -1.57079632679 -> xyz=0.0 0.0 0.144 rpy=0.0 0.0 0
- joint left_base_joint: origin xyz=0 0 0 rpy=0 0 3.141592653589793 -> xyz=0 0 0 rpy=0 0 0; parent left_arm_mount -> left_world
- joint left_robotiq_85_base_joint: origin xyz=0.0 0.0 0.0 rpy=0.0 0.0 1.57 -> xyz=0.0 0.0 0.0 rpy=0.0 0.0 0.0
- joint left_robotiq_85_left_finger_tip_joint: limit (none) -> lower=0.0 upper=0.8 effort=50 velocity=0.5; type continuous -> revolute
- joint left_robotiq_85_left_inner_knuckle_joint: limit (none) -> lower=0.0 upper=0.8 effort=50 velocity=0.5; type continuous -> revolute
- joint left_robotiq_85_right_finger_tip_joint: limit (none) -> lower=0.0 upper=0.8 effort=50 velocity=0.5; type continuous -> revolute
- joint left_robotiq_85_right_inner_knuckle_joint: limit (none) -> lower=0.0 upper=0.8 effort=50 velocity=0.5; type continuous -> revolute
- joint r_gripper_tool_frame_joint: origin xyz=0.0 0.0 0.144 rpy=0.0 -1.57079632679 -1.57079632679 -> xyz=0.0 0.0 0.144 rpy=0.0 0.0 0
- joint right_base_joint: parent right_arm_mount -> right_world
- joint right_robotiq_85_base_joint: origin xyz=0.0 0.0 0.0 rpy=0.0 0.0 1.57 -> xyz=0.0 0.0 0.0 rpy=0.0 0.0 0.0
- joint right_robotiq_85_left_finger_tip_joint: limit (none) -> lower=0.0 upper=0.8 effort=50 velocity=0.5; type continuous -> revolute
- joint right_robotiq_85_left_inner_knuckle_joint: limit (none) -> lower=0.0 upper=0.8 effort=50 velocity=0.5; type continuous -> revolute
- joint right_robotiq_85_right_finger_tip_joint: limit (none) -> lower=0.0 upper=0.8 effort=50 velocity=0.5; type continuous -> revolute
- joint right_robotiq_85_right_inner_knuckle_joint: limit (none) -> lower=0.0 upper=0.8 effort=50 velocity=0.5; type continuous -> revolute
- joint table_joint: origin xyz=0.0 0.0 0.0 rpy=0.0 0.0 0.0 -> xyz=0.0 0.0 0.88 rpy=0.0 0.0 0.0; parent world -> map
